File: hardware/kicad/native/PCB-MIC/PCB-MIC.kicad_pcb (KiCad board)
At the start: 2 copper layers, 24 x 22 mm, 6 parts, among them J1 5040500691

Commit message: hardware: shorten PCB-MIC decoupling return
Routing:
- net GND: track 35.2 -> 32.4 mm
- removed copper zone on B.Cu, net GND
Changed lines of the file:
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@@
 	)
 	(segment
-		(start 9 13.25)
-		(end 15.25 13.25)
+		(start 15.25 13.25)
+		(end 15 16.649999)
 		(width 0.5)
 		(layer "B.Cu")
@@
 		(net 7)
 	)
-	(zone
-		(net 2)
-		(net_name "GND")
-		(layer "B.Cu")
-		(name "PCB_MIC_BCU_GND_REFERENCE")
-		(hatch edge 0.5)
-		(connect_pads
-			(clearance 0.5)
-		)
-		(min_thickness 0.25)
-		(filled_areas_thickness no)
-		(fill
-			(thermal_gap 0.5)
-			(thermal_bridge_width 0.5)
-		)
-		(polygon
-			(pts
-				(xy 0.65 0.65) (xy 23.35 0.65) (xy 23.35 21.35) (xy 0.65 21.35)
-			)
-		)
-	)
 	(embedded_fonts no)
