File: hardware/kicad/native/PCB-MIC/PCB-MIC.kicad_pcb (KiCad board)
At the start: 2 copper layers, 24 x 22 mm, 6 parts, among them J1 5040500691

Commit message: Fix PCB-MIC KiCad Altium connectivity parity
Parts:
- C1: footprint C_0402_1005Metric -> Capacitor_SMD:C_0402_1005Metric
- MK1: value T5838 -> MMICT5838-00-012
- R1: footprint R_0402_1005Metric -> Resistor_SMD:R_0402_1005Metric
Connections:
- net 1V8_MIC renamed /1V8_MIC
- net AAD_CFG renamed /AAD_CFG
- net GND renamed /GND
- net MIC_WAKE renamed /MIC_WAKE
- net PDM_CLK renamed /PDM_CLK
- net PDM_DATA renamed /PDM_DATA
- net PDM_DATA_MIC renamed /PDM_DATA_MIC
Changed lines of the file:
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@@
 	)
 	(net 0 "")
-	(net 1 "1V8_MIC")
-	(net 2 "GND")
-	(net 3 "PDM_CLK")
-	(net 4 "PDM_DATA")
-	(net 5 "MIC_WAKE")
-	(net 6 "AAD_CFG")
-	(net 7 "PDM_DATA_MIC")
+	(net 1 "/1V8_MIC")
+	(net 2 "/GND")
+	(net 3 "/PDM_CLK")
+	(net 4 "/PDM_DATA")
+	(net 5 "/MIC_WAKE")
+	(net 6 "/AAD_CFG")
+	(net 7 "/PDM_DATA_MIC")
 	(footprint "Dioneya:T5838_RevA"
 		(layer "F.Cu")
@@
 			)
 		)
-		(property "Value" "T5838"
+		(property "Value" "MMICT5838-00-012"
 			(at 0 0 0)
 			(layer "F.Fab")
@@
 			)
 		)
-		(property "Datasheet" ""
+		(property "Datasheet" "TDK DS-000383 v1.2"
 			(at 0 0 0)
 			(layer "F.Fab")
@@
 			(size 0.522 0.725)
 			(layers "F.Cu" "F.Mask" "F.Paste")
-			(net 7 "PDM_DATA_MIC")
+			(net 7 "/PDM_DATA_MIC")
 			(solder_paste_margin -0.05)
 			(thermal_bridge_angle 45)
@@
 			(size 0.522 0.725)
 			(layers "F.Cu" "F.Mask" "F.Paste")
-			(net 2 "GND")
+			(net 2 "/GND")
 			(solder_paste_margin -0.05)
 			(thermal_bridge_angle 45)
@@
 			(size 0.145691 0.3)
 			(layers "F.Cu" "F.Mask")
-			(net 2 "GND")
+			(net 2 "/GND")
 			(thermal_bridge_angle 45)
 		)
@@
 			(size 0.145691 0.3)
 			(layers "F.Cu" "F.Mask")
-			(net 2 "GND")
+			(net 2 "/GND")
 			(thermal_bridge_angle 45)
 		)
@@
 			(size 0.145691 0.3)
 			(layers "F.Cu" "F.Mask")
-			(net 2 "GND")
+			(net 2 "/GND")
 			(thermal_bridge_angle 45)
 		)
@@
 			(size 0.145691 0.3)
 			(layers "F.Cu" "F.Mask")
-			(net 2 "GND")
+			(net 2 "/GND")
 			(thermal_bridge_angle 45)
 		)
@@
 			(size 0.145691 0.3)
 			(layers "F.Cu" "F.Mask")
-			(net 2 "GND")
+			(net 2 "/GND")
 			(thermal_bridge_angle 45)
 		)
@@
 			(size 0.145691 0.3)
 			(layers "F.Cu" "F.Mask")
-			(net 2 "GND")
+			(net 2 "/GND")
 			(thermal_bridge_angle 45)
 		)
@@
 			(size 0.145691 0.3)
 			(layers "F.Cu" "F.Mask")
-			(net 2 "GND")
+			(net 2 "/GND")
 			(thermal_bridge_angle 45)
 		)
@@
 			(size 0.145691 0.3)
 			(layers "F.Cu" "F.Mask")
-			(net 2 "GND")
+			(net 2 "/GND")
 			(thermal_bridge_angle 45)
 		)
@@
 			(size 0.145691 0.3)
 			(layers "F.Cu" "F.Mask")
-			(net 2 "GND")
+			(net 2 "/GND")
 			(thermal_bridge_angle 45)
 		)
@@
 			(size 0.145691 0.3)
 			(layers "F.Cu" "F.Mask")
-			(net 2 "GND")
+			(net 2 "/GND")
 			(thermal_bridge_angle 45)
 		)
@@
 			(size 0.145691 0.3)
 			(layers "F.Cu" "F.Mask")
-			(net 2 "GND")
+			(net 2 "/GND")
 			(thermal_bridge_angle 45)
 		)
@@
 			(size 0.145691 0.3)
 			(layers "F.Cu" "F.Mask")
-			(net 2 "GND")
+			(net 2 "/GND")
 			(thermal_bridge_angle 45)
 		)
@@
 			(size 0.145691 0.3)
 			(layers "F.Cu" "F.Mask")
-			(net 2 "GND")
+			(net 2 "/GND")
 			(thermal_bridge_angle 45)
 		)
@@
 			(size 0.145691 0.3)
 			(layers "F.Cu" "F.Mask")
-			(net 2 "GND")
+			(net 2 "/GND")
 			(thermal_bridge_angle 45)
 		)
@@
 			(size 0.145691 0.3)
 			(layers "F.Cu" "F.Mask")
-			(net 2 "GND")
+			(net 2 "/GND")
 			(thermal_bridge_angle 45)
 		)
@@
 			(size 0.145691 0.3)
 			(layers "F.Cu" "F.Mask")
-			(net 2 "GND")
+			(net 2 "/GND")
 			(thermal_bridge_angle 45)
 		)
@@
 			(size 0.145691 0.3)
 			(layers "F.Cu" "F.Mask")
-			(net 2 "GND")
+			(net 2 "/GND")
 			(thermal_bridge_angle 45)
 		)
@@
 			(size 0.145691 0.3)
 			(layers "F.Cu" "F.Mask")
-			(net 2 "GND")
+			(net 2 "/GND")
 			(thermal_bridge_angle 45)
 		)
@@
 			(size 0.145691 0.3)
 			(layers "F.Cu" "F.Mask")
-			(net 2 "GND")
+			(net 2 "/GND")
 			(thermal_bridge_angle 45)
 		)
@@
 			(size 0.145691 0.3)
 			(layers "F.Cu" "F.Mask")
-			(net 2 "GND")
+			(net 2 "/GND")
 			(thermal_bridge_angle 45)
 		)
@@
 			(size 0.145691 0.3)
 			(layers "F.Cu" "F.Mask")
-			(net 2 "GND")
+			(net 2 "/GND")
 			(thermal_bridge_angle 45)
 		)
@@
 			(size 0.145691 0.3)
 			(layers "F.Cu" "F.Mask")
-			(net 2 "GND")
+			(net 2 "/GND")
 			(thermal_bridge_angle 45)
 		)
@@
 			(size 0.145691 0.3)
 			(layers "F.Cu" "F.Mask")
-			(net 2 "GND")
+			(net 2 "/GND")
 			(thermal_bridge_angle 45)
 		)
@@
 			(size 0.145691 0.3)
 			(layers "F.Cu" "F.Mask")
-			(net 2 "GND")
+			(net 2 "/GND")
 			(thermal_bridge_angle 45)
 		)
@@
 			(size 0.145691 0.3)
 			(layers "F.Cu" "F.Mask")
-			(net 2 "GND")
+			(net 2 "/GND")
 			(thermal_bridge_angle 45)
 		)
@@
 			(size 0.145691 0.3)
 			(layers "F.Cu" "F.Mask")
-			(net 2 "GND")
+			(net 2 "/GND")
 			(thermal_bridge_angle 45)
 		)
@@
 			(size 0.145691 0.3)
 			(layers "F.Cu" "F.Mask")
-			(net 2 "GND")
+			(net 2 "/GND")
 			(thermal_bridge_angle 45)
 		)
@@
 			(size 0.145691 0.3)
 			(layers "F.Cu" "F.Mask")
-			(net 2 "GND")
+			(net 2 "/GND")
 			(thermal_bridge_angle 45)
 		)
@@
 			(size 0.145691 0.3)
 			(layers "F.Cu" "F.Mask")
-			(net 2 "GND")
+			(net 2 "/GND")
 			(thermal_bridge_angle 45)
 		)
@@
 			(size 0.145691 0.3)
 			(layers "F.Cu" "F.Mask")
-			(net 2 "GND")
+			(net 2 "/GND")
 			(thermal_bridge_angle 45)
 		)
@@
 			(size 0.145691 0.3)
 			(layers "F.Cu" "F.Mask")
-			(net 2 "GND")
+			(net 2 "/GND")
 			(thermal_bridge_angle 45)
 		)
@@
 			(size 0.145691 0.3)
 			(layers "F.Cu" "F.Mask")
-			(net 2 "GND")
+			(net 2 "/GND")
 			(thermal_bridge_angle 45)
 		)
@@
 			(size 0.3 0.3)
 			(layers "F.Cu" "F.Mask" "F.Paste")
-			(net 5 "MIC_WAKE")
+			(net 5 "/MIC_WAKE")
 			(solder_paste_margin -0.015)
 			(thermal_bridge_angle 45)
@@
 			(size 0.3 0.3)
 			(layers "F.Cu" "F.Mask" "F.Paste")
-			(net 6 "AAD_CFG")
+			(net 6 "/AAD_CFG")
 			(solder_paste_margin -0.015)
 			(thermal_bridge_angle 45)
@@
 			(size 0.522 0.725)
 			(layers "F.Cu" "F.Mask" "F.Paste")
-			(net 3 "PDM_CLK")
+			(net 3 "/PDM_CLK")
 			(solder_paste_margin -0.05)
 			(thermal_bridge_angle 45)
@@
 			(size 0.522 0.725)
 			(layers "F.Cu" "F.Mask" "F.Paste")
-			(net 1 "1V8_MIC")
+			(net 1 "/1V8_MIC")
 			(solder_paste_margin -0.05)
 			(thermal_bridge_angle 45)
@@
 		(embedded_fonts no)
 	)
-	(footprint "C_0402_1005Metric"
+	(footprint "Capacitor_SMD:C_0402_1005Metric"
 		(layer "F.Cu")
 		(at 14.1 13.25)
@@
 			(layers "F.Cu" "F.Mask" "F.Paste")
 			(roundrect_rratio 0.25)
-			(net 1 "1V8_MIC")
+			(net 1 "/1V8_MIC")
 		)
 		(pad "2" smd roundrect
@@
 			(layers "F.Cu" "F.Mask" "F.Paste")
 			(roundrect_rratio 0.25)
-			(net 2 "GND")
+			(net 2 "/GND")
 		)
 		(embedded_fonts no)
@@
 			)
 		)
-		(property "Datasheet" ""
+		(property "Datasheet" "Molex 504050 series"
 			(at 0 0 180)
 			(layer "F.Fab")
@@
 			(size 0.6 1)
 			(layers "F.Cu" "F.Mask" "F.Paste")
-			(net 1 "1V8_MIC")
+			(net 1 "/1V8_MIC")
 			(solder_paste_margin 0)
 		)
@@
 			(size 0.6 1)
 			(layers "F.Cu" "F.Mask" "F.Paste")
-			(net 2 "GND")
+			(net 2 "/GND")
 			(solder_paste_margin 0)
 		)
@@
 			(size 0.6 1)
 			(layers "F.Cu" "F.Mask" "F.Paste")
-			(net 3 "PDM_CLK")
+			(net 3 "/PDM_CLK")
 			(solder_paste_margin 0)
 		)
@@
 			(size 0.6 1)
 			(layers "F.Cu" "F.Mask" "F.Paste")
-			(net 4 "PDM_DATA")
+			(net 4 "/PDM_DATA")
 			(solder_paste_margin 0)
 		)
@@
 			(size 0.6 1)
 			(layers "F.Cu" "F.Mask" "F.Paste")
-			(net 5 "MIC_WAKE")
+			(net 5 "/MIC_WAKE")
 			(solder_paste_margin 0)
 		)
@@
 			(size 0.6 1)
 			(layers "F.Cu" "F.Mask" "F.Paste")
-			(net 6 "AAD_CFG")
+			(net 6 "/AAD_CFG")
 			(solder_paste_margin 0)
 		)
@@
 		)
 	)
-	(footprint "R_0402_1005Metric"
+	(footprint "Resistor_SMD:R_0402_1005Metric"
 		(layer "F.Cu")
 		(at 11.25 10.55 -90)
@@
 			(layers "F.Cu" "F.Mask" "F.Paste")
 			(roundrect_rratio 0.25)
-			(net 4 "PDM_DATA")
+			(net 4 "/PDM_DATA")
 		)
 		(pad "2" smd roundrect
@@
 			(layers "F.Cu" "F.Mask" "F.Paste")
 			(roundrect_rratio 0.25)
-			(net 7 "PDM_DATA_MIC")
+			(net 7 "/PDM_DATA_MIC")
 		)
 		(embedded_fonts no)
