File: hardware/kicad/native/PCB-MAIN/PCB-MAIN.kicad_pcb (KiCad board)
At the start: 6 copper layers, 110 x 75 mm, 251 parts, among them J10 U.FL-R-SMT-1(60), J11 USB4105-GF-A-120, J12 MEM2052-00-195-00-A, J13 504050-0291, J6 2336582-1, J7 2336582-1, J8 U.FL-R-SMT-1(60), J9 U.FL-R-SMT-1(60), Q1 MMBT3904,215, Q2 MMBT3904,215, Q3 MMBT3904,215, Q4 Si1016X-T1-GE3, U1 STM32U585VIT6Q, U10 E22-900M22S, U11 MDBT50Q-P1MV2, U13 TS3A27518EPWR, U14 ESDALC6V1-5P6, U15 ESDALC6V1-5P6, U16 SN74AXC8T245PWR, U17 SN74LVC32APWR, U18 SN74AXC1T45DRLR, U19 TPD4E05U06DQAR, U2 W25Q512JVFIQ, U20 TPD4E05U06DQAR, U21 TPD4E05U06DQAR, U22 TPD4E05U06DQAR, U23 TPD4E05U06DQAR, U24 TPD4E05U06DQAR, U25 TPD2EUSB30DRTR, U26 TPD2EUSB30DRTR, U27 TPD4E05U06DQAR, U3 LIS2DW12TR, U4 STTS22HTR, U5 LT6000IDCB#TRMPBF, U6 SN74LVC1G07DBVR, U7 SN74AXC8T245PWR, U8 BG95-M3, U9 MAX-M10S-00B, X1 SiT1552AI-JE-DCC-32.768D

Commit message: pcb(main): control TI DBV SOT23-5 land pattern
Parts:
- U6: footprint SOT-23-5 -> TI_DBV0005A_SOT23-5
Changed lines of the file:
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@@
       (net 129 "SD_CMD_CARD") (thermal_bridge_angle 45))
   )
-  (footprint "SOT-23-5" (layer "F.Cu")
+  (footprint "TI_DBV0005A_SOT23-5" (version 20221018) (generator pcbnew) (layer "F.Cu")
     (at 46 41)
-    (descr "SOT, 5 Pin (https://www.jedec.org/sites/default/files/docs/Mo-178c.PDF variant AA), generated with kicad-footprint-generator ipc_gullwing_generator.py")
-    (tags "SOT TO_SOT_SMD")
-    (property "DIONEA_FOOTPRINT_SOURCE" "KiCad:Package_TO_SOT_SMD.pretty/SOT-23-5")
-    (property "DIONEA_FOOTPRINT_STATUS" "KICAD_LIBRARY_PATTERN_REVIEW_PENDING")
+    (descr "TI DBV0005A 5-pin SOT-23; 4214839/K 08/2024 example board layout")
+    (tags "Texas Instruments DBV0005A SOT-23-5 0.95mm")
+    (property "DIONEA_FOOTPRINT_SOURCE" "TI_DBV0005A_4214839K_2024-08_RecommendedLandPattern")
+    (property "DIONEA_FOOTPRINT_STATUS" "MANUFACTURER_DRAWING_PATTERN_CONTROLLED")
     (property "DIONEA_PACKAGE" "SOT-23-5_DBV")
     (property "DIONEA_POPULATION" "FITTED")
     (attr smd)
+    (fp_rect (start -2.1 -1.78) (end 2.1 1.78) (layer "F.CrtYd") (stroke (width 0.05) (type default)) (fill none))
+    (fp_poly (pts
+        (xy -0.8 -1.05)
+        (xy -0.4 -1.45)
+        (xy 0.8 -1.45)
+        (xy 0.8 1.45)
+        (xy -0.8 1.45)
+      ) (layer "F.Fab") (stroke (width 0.1) (type default)) (fill none))
+    (fp_poly (pts
+        (xy -1.48 -1.08)
+        (xy -1.68 -1.28)
+        (xy -1.28 -1.28)
+      ) (layer "F.SilkS") (stroke (width 0.12) (type default)) (fill solid))
     (fp_text reference "U6" (at 0 -1.2) (layer "F.SilkS")
-        (effects (font (size 0.8 0.8) (thickness 0.12)))
+      (effects (font (size 0.8 0.8) (thickness 0.12)))
     )
     (fp_text value "SN74LVC1G07DBVR" (at 0 2.4) (layer "F.Fab") hide
-        (effects (font (size 1 1) (thickness 0.15)))
+      (effects (font (size 1 1) (thickness 0.15)))
     )
-    (fp_text user "${REFERENCE}" (at 0 0) (layer "F.Fab")
-        (effects (font (size 0.4 0.4) (thickness 0.06)))
-    )
-    (fp_line (start 0 -1.56) (end -0.8 -1.56)
-      (stroke (width 0.12) (type solid)) (layer "F.SilkS"))
-    (fp_line (start 0 -1.56) (end 0.8 -1.56)
-      (stroke (width 0.12) (type solid)) (layer "F.SilkS"))
-    (fp_line (start 0 1.56) (end -0.8 1.56)
-      (stroke (width 0.12) (type solid)) (layer "F.SilkS"))
-    (fp_line (start 0 1.56) (end 0.8 1.56)
-      (stroke (width 0.12) (type solid)) (layer "F.SilkS"))
-    (fp_poly
-      (pts
-        (xy -1.3 -1.51)
-        (xy -1.54 -1.84)
-        (xy -1.06 -1.84)
-        (xy -1.3 -1.51)
-      )
-      (stroke (width 0.12) (type solid)) (fill solid) (layer "F.SilkS"))
-    (fp_line (start -2.05 -1.7) (end -2.05 1.7)
-      (stroke (width 0.05) (type solid)) (layer "F.CrtYd"))
-    (fp_line (start -2.05 1.7) (end 2.05 1.7)
-      (stroke (width 0.05) (type solid)) (layer "F.CrtYd"))
-    (fp_line (start 2.05 -1.7) (end -2.05 -1.7)
-      (stroke (width 0.05) (type solid)) (layer "F.CrtYd"))
-    (fp_line (start 2.05 1.7) (end 2.05 -1.7)
-      (stroke (width 0.05) (type solid)) (layer "F.CrtYd"))
-    (fp_line (start -0.8 -1.05) (end -0.4 -1.45)
-      (stroke (width 0.1) (type solid)) (layer "F.Fab"))
-    (fp_line (start -0.8 1.45) (end -0.8 -1.05)
-      (stroke (width 0.1) (type solid)) (layer "F.Fab"))
-    (fp_line (start -0.4 -1.45) (end 0.8 -1.45)
-      (stroke (width 0.1) (type solid)) (layer "F.Fab"))
-    (fp_line (start 0.8 -1.45) (end 0.8 1.45)
-      (stroke (width 0.1) (type solid)) (layer "F.Fab"))
-    (fp_line (start 0.8 1.45) (end -0.8 1.45)
-      (stroke (width 0.1) (type solid)) (layer "F.Fab"))
-    (pad "1" smd roundrect (at -1.1375 -0.95) (size 1.325 0.6) (layers "F.Cu" "F.Paste" "F.Mask") (roundrect_rratio 0.25))
-    (pad "2" smd roundrect (at -1.1375 0) (size 1.325 0.6) (layers "F.Cu" "F.Paste" "F.Mask") (roundrect_rratio 0.25)
-      (net 11 "BLE_EN"))
-    (pad "3" smd roundrect (at -1.1375 0.95) (size 1.325 0.6) (layers "F.Cu" "F.Paste" "F.Mask") (roundrect_rratio 0.25)
-      (net 45 "GND_DIGITAL"))
-    (pad "4" smd roundrect (at 1.1375 0.95) (size 1.325 0.6) (layers "F.Cu" "F.Paste" "F.Mask") (roundrect_rratio 0.25)
-      (net 105 "NRF_RESET_N"))
-    (pad "5" smd roundrect (at 1.1375 -0.95) (size 1.325 0.6) (layers "F.Cu" "F.Paste" "F.Mask") (roundrect_rratio 0.25)
-      (net 2 "3V3_DIGITAL"))
-    (model "${KICAD7_3DMODEL_DIR}/Package_TO_SOT_SMD.3dshapes/SOT-23-5.wrl"
-      (offset (xyz 0 0 0))
-      (scale (xyz 1 1 1))
-      (rotate (xyz 0 0 0))
-    )
+    (pad "1" smd roundrect (at -1.3 -0.95) (size 1.1 0.6) (layers "F.Cu" "F.Paste" "F.Mask") (roundrect_rratio 0.166667)
+      (solder_mask_margin 0.07))
+    (pad "2" smd roundrect (at -1.3 0) (size 1.1 0.6) (layers "F.Cu" "F.Paste" "F.Mask") (roundrect_rratio 0.166667)
+      (net 11 "BLE_EN") (solder_mask_margin 0.07))
+    (pad "3" smd roundrect (at -1.3 0.95) (size 1.1 0.6) (layers "F.Cu" "F.Paste" "F.Mask") (roundrect_rratio 0.166667)
+      (net 45 "GND_DIGITAL") (solder_mask_margin 0.07))
+    (pad "4" smd roundrect (at 1.3 0.95) (size 1.1 0.6) (layers "F.Cu" "F.Paste" "F.Mask") (roundrect_rratio 0.166667)
+      (net 105 "NRF_RESET_N") (solder_mask_margin 0.07))
+    (pad "5" smd roundrect (at 1.3 -0.95) (size 1.1 0.6) (layers "F.Cu" "F.Paste" "F.Mask") (roundrect_rratio 0.166667)
+      (net 2 "3V3_DIGITAL") (solder_mask_margin 0.07))
   )
   (footprint "" (layer "F.Cu")

Commit message: pcb(main): control ST SOT666 land pattern
Parts:
- U14, U15: footprint SOT-666 -> ST_ESDALC6V1-5P6_SOT666
