File: hardware/kicad/native/PCB-MAIN/PCB-MAIN.kicad_sch (KiCad schematic)
At the start: 248 parts, among them J10 U.FL-R-SMT-1(60), J11 USB4105-GF-A-120, J12 MEM2052-00-195-00-A, J13 504050-0291, J6 2336582-1, J7 2336582-1, J8 U.FL-R-SMT-1(60), J9 U.FL-R-SMT-1(60), Q1 MMBT3904,215, Q2 MMBT3904,215, Q3 MMBT3904,215, Q4 Complementary N and P channel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, U1 STM32U585VIT6Q, U10 E22-900M22S, U11 MDBT50Q-P1MV2, U12 SDCIT2/32GB, U13 TS3A27518EPWR, U14 ESDALC6V1-5P6, U15 ESDALC6V1-5P6, U16 SN74AXC8T245PWR, U17 SN74LVC32APWR, U18 SN74AXC1T45DRLR, U19 4 channel 0.5 pF ESD, U2 W25Q512JVFIQ, U20 4 channel 0.5 pF ESD, U21 4 channel 0.5 pF ESD, U22 4 channel 0.5 pF ESD, U23 4 channel 0.5 pF ESD, U24 4 channel 0.5 pF ESD, U25 2 channel 0.7 pF USB ESD, U26 2 channel 0.7 pF USB ESD, U27 4 channel 0.5 pF ESD, U3 LIS2DW12TR, U4 STTS22HTR, U5 Single rail-to-rail low-power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, U6 Single non-inverting open-dra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, U7 SN74AXC8T245PWR, U8 BG95-M3, U9 MAX-M10S-00B, X1 32.768 kHz full-swing LVCMOS

Commit message: fix(pcb-main): make native ERC inputs deterministic
Parts:
- C36, C44: footprint DioneyaMain:7343-31 -> (none)
- D1, D2: footprint DioneyaMain:SOD882 -> (none)
- D10, D11, D4, D6, D7, D8, D9: footprint DioneyaMain:SOD-523_DYA -> (none)
- D3, D5: footprint DioneyaMain:SOD962-2 -> (none)
- FL1: footprint DioneyaMain:1109-5 -> (none)
- J10, J8, J9: footprint DioneyaMain:U.FL_SMT -> (none)
- J11: footprint DioneyaMain:USB-C_16P_horizontal_top_mount_1.20mm_stake -> (none)
- J12: footprint DioneyaMain:microSD_push-push_1.95mm_8P_CD -> (none)
- J13: footprint DioneyaMain:Pico-Lock_1.5mm_2P_RA_SMT -> (none)
- J6, J7: footprint DioneyaMain:TE_NanoSIM_H1.37 -> (none)
- J_MIC1, J_MIC2, J_MIC3, J_MIC4: footprint DioneyaMain:Pico-Lock_1.5_1x06_Right_Angle -> (none)
- J_PWR: footprint DioneyaMain:Micro-Fit_3.0_2x06_Right_Angle -> (none)
- Q1, Q2, Q3: footprint DioneyaMain:SOT23 -> (none)
- Q4: footprint DioneyaMain:SOT-563_SC-89 -> (none)
- TP_BLE_SWD, TP_CELL_USB: footprint DioneyaMain:POGO_FIXTURE_4P -> (none)
- TP_CELL_DBG, TP_MCU_SWD: footprint DioneyaMain:POGO_FIXTURE_5P -> (none)
- TP_EOL: footprint DioneyaMain:POGO_FIXTURE_13P -> (none)
- U1: footprint DioneyaMain:LQFP100_14x14 -> (none)
- U10: footprint DioneyaMain:SMD_20x14_22P_1.27mm -> (none)
- U11: footprint DioneyaMain:nRF52840_SMD_10.5x15.5_61P_PCB_antenna -> (none)
- U13, U16, U7: footprint DioneyaMain:TSSOP-24_PW -> (none)
- U14, U15: footprint DioneyaMain:SOT666_1.6x1.6mm -> (none)
- U17: footprint DioneyaMain:TSSOP-14_PW -> (none)
- U18: footprint DioneyaMain:SOT-5X3-6_DRL -> (none)
- U19, U20, U21, U22, U23, U24, U27: footprint DioneyaMain:USON-10_DQA -> (none)
- U2: footprint DioneyaMain:SOIC-16_300mil_F -> (none)
- U25, U26: footprint DioneyaMain:SOT-9X3_DRT -> (none)
- U3: footprint DioneyaMain:LGA-12_2x2mm -> (none)
- U4: footprint DioneyaMain:UDFN-6L_2x2mm -> (none)
- U5: footprint DioneyaMain:DFN-6_DCB_2x3mm -> (none)
- U6: footprint DioneyaMain:SOT-23-5_DBV -> (none)
- U8: footprint DioneyaMain:LGA-102_23.6x19.9mm -> (none)
- U9: footprint DioneyaMain:LCC-18_9.7x10.1mm -> (none)
- X1: footprint DioneyaMain:CSP-4_1.5x0.8mm -> (none)
Other:
- moved on the sheet: C1, C10, C11, C12, C13, C14, C15, C17, C2, C21, C23, C25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

Commit message: hardware: materialize PCB-MAIN hierarchy and pad nets
Parts:
- removed C1: 100 nF 25 V X7R, Capacitor_SMD:C_0402_1005Metric, symbol DioneyaMain:C1_GRM155R71E104KE14D
- removed C10: 100 nF 25 V X7R, Capacitor_SMD:C_0402_1005Metric, symbol DioneyaMain:C10_GRM155R71E104KE14D
- removed C11: 1 uF 16 V X5R, Capacitor_SMD:C_0402_1005Metric, symbol DioneyaMain:C11_GRM155R61C105KA12D
- removed C12: 100 nF 25 V X7R, Capacitor_SMD:C_0402_1005Metric, symbol DioneyaMain:C12_GRM155R71E104KE14D
- removed C13: 10 uF 10 V X5R, Capacitor_SMD:C_0603_1608Metric, symbol DioneyaMain:C13_GRM188R61A106KE69D
- removed C14: 2.2 uF 10 V X5R, Capacitor_SMD:C_0402_1005Metric, symbol DioneyaMain:C14_GRM155R61A225KE15D
- removed C15: 2.2 uF 10 V X5R, Capacitor_SMD:C_0402_1005Metric, symbol DioneyaMain:C15_GRM155R61A225KE15D
- removed C16: 100 nF 25 V X7R, Capacitor_SMD:C_0402_1005Metric, symbol DioneyaMain:C16_GRM155R71E104KE14D
- removed C17: 100 nF 25 V X7R, Capacitor_SMD:C_0402_1005Metric, symbol DioneyaMain:C17_GRM155R71E104KE14D
- removed C18: 100 nF 25 V X7R, Capacitor_SMD:C_0402_1005Metric, symbol DioneyaMain:C18_GRM155R71E104KE14D
- removed C19: 22 uF 10 V X5R, Capacitor_SMD:C_0805_2012Metric, symbol DioneyaMain:C19_GRM21BR61A226ME44L
- removed C2: 100 nF 25 V X7R, Capacitor_SMD:C_0402_1005Metric, symbol DioneyaMain:C2_GRM155R71E104KE14D
- removed C20: 10 uF 10 V X5R, Capacitor_SMD:C_0603_1608Metric, symbol DioneyaMain:C20_GRM188R61A106KE69D
- removed C21: 100 nF 25 V X7R, Capacitor_SMD:C_0402_1005Metric, symbol DioneyaMain:C21_GRM155R71E104KE14D
- removed C22: 1 uF 16 V X5R, Capacitor_SMD:C_0402_1005Metric, symbol DioneyaMain:C22_GRM155R61C105KA12D
- removed C23: 100 nF 25 V X7R, Capacitor_SMD:C_0402_1005Metric, symbol DioneyaMain:C23_GRM155R71E104KE14D
- removed C24: 10 uF 10 V X5R, Capacitor_SMD:C_0603_1608Metric, symbol DioneyaMain:C24_GRM188R61A106KE69D
- removed C25: 100 nF 25 V X7R, Capacitor_SMD:C_0402_1005Metric, symbol DioneyaMain:C25_GRM155R71E104KE14D
- removed C26: 100 nF 25 V X7R, Capacitor_SMD:C_0402_1005Metric, symbol DioneyaMain:C26_GRM155R71E104KE14D
- removed C27: 100 nF 25 V X7R, Capacitor_SMD:C_0402_1005Metric, symbol DioneyaMain:C27_GRM155R71E104KE14D
- removed C28: 100 nF 25 V X7R, Capacitor_SMD:C_0402_1005Metric, symbol DioneyaMain:C28_GRM155R71E104KE14D
- removed C29: 100 nF 25 V X7R, Capacitor_SMD:C_0402_1005Metric, symbol DioneyaMain:C29_GRM155R71E104KE14D
- removed C3: 100 nF 25 V X7R, Capacitor_SMD:C_0402_1005Metric, symbol DioneyaMain:C3_GRM155R71E104KE14D
- removed C30: 100 nF 25 V X7R, Capacitor_SMD:C_0402_1005Metric, symbol DioneyaMain:C30_GRM155R71E104KE14D
- removed C31: 100 nF 25 V X7R, Capacitor_SMD:C_0402_1005Metric, symbol DioneyaMain:C31_GRM155R71E104KE14D
- removed C32: 100 nF 25 V X7R, Capacitor_SMD:C_0402_1005Metric, symbol DioneyaMain:C32_GRM155R71E104KE14D
- removed C33: 100 nF 25 V X7R, Capacitor_SMD:C_0402_1005Metric, symbol DioneyaMain:C33_GRM155R71E104KE14D
- removed C34: 100 nF 25 V X7R, Capacitor_SMD:C_0402_1005Metric, symbol DioneyaMain:C34_GRM155R71E104KE14D
- removed C35: 100 nF 25 V X7R, Capacitor_SMD:C_0402_1005Metric, symbol DioneyaMain:C35_GRM155R71E104KE14D
- removed C36: 100 uF 6.3 V 15 mOhm polymer, symbol DioneyaMain:C36_T520D107M006ATE015
- removed C37: 220 nF 25 V X7R, Capacitor_SMD:C_0402_1005Metric, symbol DioneyaMain:C37_GRM155R71E224KE14D
- removed C38: 47 nF 25 V X7R, Capacitor_SMD:C_0402_1005Metric, symbol DioneyaMain:C38_GRM155R71E473KA01D
- removed C39: 150 pF 50 V C0G, Capacitor_SMD:C_0402_1005Metric, symbol DioneyaMain:C39_GRM1555C1H151JA01D
- removed C4: 100 nF 25 V X7R, Capacitor_SMD:C_0402_1005Metric, symbol DioneyaMain:C4_GRM155R71E104KE14D
- removed C40: 100 pF 50 V C0G, Capacitor_SMD:C_0402_1005Metric, symbol DioneyaMain:C40_GRM1555C1H101JA01D
- removed C41: 68 pF 50 V C0G, Capacitor_SMD:C_0402_1005Metric, symbol DioneyaMain:C41_GRM1555C1H680JA01D
- removed C42: 33 pF 50 V C0G, Capacitor_SMD:C_0402_1005Metric, symbol DioneyaMain:C42_GRM1555C1H330JA01D
- removed C43: 10 pF 50 V C0G, Capacitor_SMD:C_0402_1005Metric, symbol DioneyaMain:C43_GRM1555C1H100JA01D
- removed C44: 100 uF 6.3 V 15 mOhm polymer, symbol DioneyaMain:C44_T520D107M006ATE015
- removed C45: 100 nF 25 V X7R, Capacitor_SMD:C_0402_1005Metric, symbol DioneyaMain:C45_GRM155R71E104KE14D
- removed C46: 33 pF 50 V C0G, Capacitor_SMD:C_0402_1005Metric, symbol DioneyaMain:C46_GRM1555C1H330JA01D
- removed C47: 10 pF 50 V C0G, Capacitor_SMD:C_0402_1005Metric, symbol DioneyaMain:C47_GRM1555C1H100JA01D
- removed C48: 10 nF 25 V X7R, Capacitor_SMD:C_0402_1005Metric, symbol DioneyaMain:C48_GRM155R71E103KA01D
- removed C49: 100 nF 25 V X7R, Capacitor_SMD:C_0402_1005Metric, symbol DioneyaMain:C49_GRM155R71E104KE14D
- removed C5: 100 nF 25 V X7R, Capacitor_SMD:C_0402_1005Metric, symbol DioneyaMain:C5_GRM155R71E104KE14D
- removed C50: 100 nF 25 V X7R, Capacitor_SMD:C_0402_1005Metric, symbol DioneyaMain:C50_GRM155R71E104KE14D
- removed C51: 100 nF 25 V X7R, Capacitor_SMD:C_0402_1005Metric, symbol DioneyaMain:C51_GRM155R71E104KE14D
- removed C52: 10 nF 25 V X7R, Capacitor_SMD:C_0402_1005Metric, symbol DioneyaMain:C52_GRM155R71E103KA01D
- removed C53: 10 nF 25 V X7R, Capacitor_SMD:C_0402_1005Metric, symbol DioneyaMain:C53_GRM155R71E103KA01D
- removed C54: 33 pF 50 V C0G, Capacitor_SMD:C_0402_1005Metric, symbol DioneyaMain:C54_GRM1555C1H330JA01D
- removed C55: 33 pF 50 V C0G, Capacitor_SMD:C_0402_1005Metric, symbol DioneyaMain:C55_GRM1555C1H330JA01D
- removed C56: 33 pF 50 V C0G, Capacitor_SMD:C_0402_1005Metric, symbol DioneyaMain:C56_GRM1555C1H330JA01D
- removed C57: 33 pF 50 V C0G, Capacitor_SMD:C_0402_1005Metric, symbol DioneyaMain:C57_GRM1555C1H330JA01D
- removed C58: 33 pF 50 V C0G, Capacitor_SMD:C_0402_1005Metric, symbol DioneyaMain:C58_GRM1555C1H330JA01D
- removed C59: 33 pF 50 V C0G, Capacitor_SMD:C_0402_1005Metric, symbol DioneyaMain:C59_GRM1555C1H330JA01D
- removed C6: 10 uF 10 V X5R, Capacitor_SMD:C_0603_1608Metric, symbol DioneyaMain:C6_GRM188R61A106KE69D
- removed C60: 100 nF 25 V X7R, Capacitor_SMD:C_0402_1005Metric, symbol DioneyaMain:C60_GRM155R71E104KE14D
- removed C61: 10 uF 10 V X5R, Capacitor_SMD:C_0603_1608Metric, symbol DioneyaMain:C61_GRM188R61A106KE69D
- removed C62: 100 nF 25 V X7R, Capacitor_SMD:C_0402_1005Metric, symbol DioneyaMain:C62_GRM155R71E104KE14D
- removed C63: 10 nF 16 V X7R, Capacitor_SMD:C_0402_1005Metric, symbol DioneyaMain:C63_GRM155R71C103KA01D
- removed C64: 47 pF 25 V C0G, Capacitor_SMD:C_0402_1005Metric, symbol DioneyaMain:C64_GRM1555C1E470JA01D
- removed C65: 100 nF 25 V X7R, Capacitor_SMD:C_0402_1005Metric, symbol DioneyaMain:C65_GRM155R71E104KE14D
- removed C66: 100 nF 25 V X7R, Capacitor_SMD:C_0402_1005Metric, symbol DioneyaMain:C66_GRM155R71E104KE14D
- removed C67: 10 uF 10 V X5R, Capacitor_SMD:C_0603_1608Metric, symbol DioneyaMain:C67_GRM188R61A106KE69D
- removed C68: 100 nF 25 V X7R, Capacitor_SMD:C_0402_1005Metric, symbol DioneyaMain:C68_GRM155R71E104KE14D
- removed C69: 10 pF 50 V C0G, Capacitor_SMD:C_0402_1005Metric, symbol DioneyaMain:C69_GRM1555C1H100JA01D
- removed C7: 100 nF 25 V X7R, Capacitor_SMD:C_0402_1005Metric, symbol DioneyaMain:C7_GRM155R71E104KE14D
- removed C70: 10 pF 50 V C0G, Capacitor_SMD:C_0402_1005Metric, symbol DioneyaMain:C70_GRM1555C1H100JA01D
- removed C71: 100 nF 25 V X7R, Capacitor_SMD:C_0402_1005Metric, symbol DioneyaMain:C71_GRM155R71E104KE14D
- removed C72: 10 uF 10 V X5R, Capacitor_SMD:C_0603_1608Metric, symbol DioneyaMain:C72_GRM188R61A106KE69D
- removed C73: 100 nF 25 V X7R, Capacitor_SMD:C_0402_1005Metric, symbol DioneyaMain:C73_GRM155R71E104KE14D
- removed C74: 100 nF 25 V X7R, Capacitor_SMD:C_0402_1005Metric, symbol DioneyaMain:C74_GRM155R71E104KE14D
- removed C75: 10 uF 10 V X5R, Capacitor_SMD:C_0603_1608Metric, symbol DioneyaMain:C75_GRM188R61A106KE69D
- removed C76: 10 nF 25 V X7R, Capacitor_SMD:C_0402_1005Metric, symbol DioneyaMain:C76_GRM155R71E103KA01D
- removed C77: 4.7 nF 100 V X7R, Capacitor_SMD:C_0402_1005Metric, symbol DioneyaMain:C77_GRM155R72A472KA01D
- removed C78: 10 nF 25 V X7R, Capacitor_SMD:C_0402_1005Metric, symbol DioneyaMain:C78_GRM155R71E103KA01D
- removed C79: 10 pF 50 V C0G, Capacitor_SMD:C_0402_1005Metric, symbol DioneyaMain:C79_GRM1555C1H100JA01D
- removed C8: 100 nF 25 V X7R, Capacitor_SMD:C_0402_1005Metric, symbol DioneyaMain:C8_GRM155R71E104KE14D
- removed C80: 10 pF 50 V C0G, Capacitor_SMD:C_0402_1005Metric, symbol DioneyaMain:C80_GRM1555C1H100JA01D
- removed C9: 1 uF 16 V X5R, Capacitor_SMD:C_0402_1005Metric, symbol DioneyaMain:C9_GRM155R61C105KA12D
- removed D1: 5 V unidirectional 150 W TVS, symbol DioneyaMain:D1_PESD5V0S1UL
- removed D10: 5.5 V 0.5 pF ESD, symbol DioneyaMain:D10_TPD1E05U06DYAR
- removed D11: 5.5 V 0.5 pF ESD, symbol DioneyaMain:D11_TPD1E05U06DYAR
- removed D2: 5 V unidirectional 150 W TVS, symbol DioneyaMain:D2_PESD5V0S1UL
- removed D3: 5 V bidirectional 0.2 pF RF ESD, symbol DioneyaMain:D3_PESD5V0C1BSF
- removed D4: 5.5 V unidirectional 0.5 pF RF ESD, symbol DioneyaMain:D4_TPD1E05U06DYAR
- removed D5: 5 V bidirectional 0.2 pF RF ESD, symbol DioneyaMain:D5_PESD5V0C1BSF
- removed D6: 5.5 V 0.5 pF ESD, symbol DioneyaMain:D6_TPD1E05U06DYAR
- removed D7: 5.5 V 0.5 pF ESD, symbol DioneyaMain:D7_TPD1E05U06DYAR
- removed D8: 5.5 V 0.5 pF ESD, symbol DioneyaMain:D8_TPD1E05U06DYAR
- removed D9: 5.5 V 0.5 pF ESD, symbol DioneyaMain:D9_TPD1E05U06DYAR
- removed FB1: 600 Ohm at 100 MHz, Inductor_SMD:L_1206_3216Metric, symbol DioneyaMain:FB1_BLM31KN601SN1L
- removed FL1: 1582.4 MHz wideband GNSS SAW, symbol DioneyaMain:FL1_ABSES5AF-L100KM
- removed J10: U.FL-R-SMT-1(60), symbol DioneyaMain:J10_U.FL-R-SMT-1_60
- removed J11: USB4105-GF-A-120, symbol DioneyaMain:J11_USB4105-GF-A-120
- removed J12: MEM2052-00-195-00-A, symbol DioneyaMain:J12_MEM2052-00-195-00-A
- removed J13: 504050-0291, symbol DioneyaMain:J13_504050-0291
- removed J6: 2336582-1, symbol DioneyaMain:J6_2336582-1
- removed J7: 2336582-1, symbol DioneyaMain:J7_2336582-1
- removed J8: U.FL-R-SMT-1(60), symbol DioneyaMain:J8_U.FL-R-SMT-1_60
- removed J9: U.FL-R-SMT-1(60), symbol DioneyaMain:J9_U.FL-R-SMT-1_60
- removed J_MIC1: 504050-0691, symbol DioneyaMain:J_MIC1_504050-0691
- removed J_MIC2: 504050-0691, symbol DioneyaMain:J_MIC2_504050-0691
- removed J_MIC3: 504050-0691, symbol DioneyaMain:J_MIC3_504050-0691
- removed J_MIC4: 504050-0691, symbol DioneyaMain:J_MIC4_504050-0691
- removed J_PWR: 43045-1202, symbol DioneyaMain:J_PWR_43045-1202
- removed L1: 2.2 uH 20%, Inductor_SMD:L_1210_3225Metric, symbol DioneyaMain:L1_LQH32PN2R2NN0L
- removed L2: 27 nH 5%, Inductor_SMD:L_0402_1005Metric, symbol DioneyaMain:L2_LQW15AN27NJ00D
- removed Q1: MMBT3904,215, symbol DioneyaMain:Q1_MMBT3904_215
- removed Q2: MMBT3904,215, symbol DioneyaMain:Q2_MMBT3904_215
- removed Q3: MMBT3904,215, symbol DioneyaMain:Q3_MMBT3904_215
- removed Q4: Complementary N and P channel 20 V, symbol DioneyaMain:Q4_Si1016X-T1-GE3
- removed R1: 10 kOhm 1%, Resistor_SMD:R_0402_1005Metric, symbol DioneyaMain:R1_ERJ-2RKF1002X
- removed R10: 22 Ohm 1%, Resistor_SMD:R_0402_1005Metric, symbol DioneyaMain:R10_ERJ-2RKF22R0X
- removed R100: 1 kOhm 1%, Resistor_SMD:R_0402_1005Metric, symbol DioneyaMain:R100_ERJ-2RKF1001X
- removed R101: 22 Ohm 1%, Resistor_SMD:R_0402_1005Metric, symbol DioneyaMain:R101_ERJ-2RKF22R0X
- removed R102: 1 kOhm 1%, Resistor_SMD:R_0402_1005Metric, symbol DioneyaMain:R102_ERJ-2RKF1001X
- removed R103: 0 Ohm, Resistor_SMD:R_0402_1005Metric, symbol DioneyaMain:R103_ERJ-2GE0R00X
- removed R11: 22 Ohm 1%, Resistor_SMD:R_0402_1005Metric, symbol DioneyaMain:R11_ERJ-2RKF22R0X
- removed R12: 22 Ohm 1%, Resistor_SMD:R_0402_1005Metric, symbol DioneyaMain:R12_ERJ-2RKF22R0X
- removed R13: 2.2 kOhm 1%, Resistor_SMD:R_0402_1005Metric, symbol DioneyaMain:R13_ERJ-2RKF2201X
- removed R14: 2.2 kOhm 1%, Resistor_SMD:R_0402_1005Metric, symbol DioneyaMain:R14_ERJ-2RKF2201X
- removed R15: 22 Ohm 1%, Resistor_SMD:R_0402_1005Metric, symbol DioneyaMain:R15_ERJ-2RKF22R0X
- removed R16: 22 Ohm 1%, Resistor_SMD:R_0402_1005Metric, symbol DioneyaMain:R16_ERJ-2RKF22R0X
- removed R17: 22 Ohm 1%, Resistor_SMD:R_0402_1005Metric, symbol DioneyaMain:R17_ERJ-2RKF22R0X
- removed R18: 22 Ohm 1%, Resistor_SMD:R_0402_1005Metric, symbol DioneyaMain:R18_ERJ-2RKF22R0X
- removed R19: 100 kOhm 1%, Resistor_SMD:R_0402_1005Metric, symbol DioneyaMain:R19_ERJ-2RKF1003X
- removed R2: 100 kOhm 1%, Resistor_SMD:R_0402_1005Metric, symbol DioneyaMain:R2_ERJ-2RKF1003X
- removed R20: 100 kOhm 1%, Resistor_SMD:R_0402_1005Metric, symbol DioneyaMain:R20_ERJ-2RKF1003X
- removed R21: 100 kOhm 1%, Resistor_SMD:R_0402_1005Metric, symbol DioneyaMain:R21_ERJ-2RKF1003X
- removed R22: 100 kOhm 1%, Resistor_SMD:R_0402_1005Metric, symbol DioneyaMain:R22_ERJ-2RKF1003X
- removed R23: 100 kOhm 1%, Resistor_SMD:R_0402_1005Metric, symbol DioneyaMain:R23_ERJ-2RKF1003X
- removed R24: 4.7 kOhm 1%, Resistor_SMD:R_0402_1005Metric, symbol DioneyaMain:R24_ERJ-2RKF4701X
- removed R25: 47 kOhm 1%, Resistor_SMD:R_0402_1005Metric, symbol DioneyaMain:R25_ERJ-2RKF4702X
- removed R26: 4.7 kOhm 1%, Resistor_SMD:R_0402_1005Metric, symbol DioneyaMain:R26_ERJ-2RKF4701X
- removed R27: 47 kOhm 1%, Resistor_SMD:R_0402_1005Metric, symbol DioneyaMain:R27_ERJ-2RKF4702X
- removed R28: 10 kOhm 1%, Resistor_SMD:R_0402_1005Metric, symbol DioneyaMain:R28_ERJ-2RKF1002X
- removed R29: 100 kOhm 1%, Resistor_SMD:R_0402_1005Metric, symbol DioneyaMain:R29_ERJ-2RKF1003X
- removed R3: 100 kOhm 1%, Resistor_SMD:R_0402_1005Metric, symbol DioneyaMain:R3_ERJ-2RKF1003X
- removed R30: 10 kOhm 1%, Resistor_SMD:R_0402_1005Metric, symbol DioneyaMain:R30_ERJ-2RKF1002X
- removed R31: 10 kOhm 1%, Resistor_SMD:R_0402_1005Metric, symbol DioneyaMain:R31_ERJ-2RKF1002X
- removed R32: 100 kOhm 1%, Resistor_SMD:R_0402_1005Metric, symbol DioneyaMain:R32_ERJ-2RKF1003X
- removed R33: 100 kOhm 1%, Resistor_SMD:R_0402_1005Metric, symbol DioneyaMain:R33_ERJ-2RKF1003X
- removed R34: 100 kOhm 1%, Resistor_SMD:R_0402_1005Metric, symbol DioneyaMain:R34_ERJ-2RKF1003X
- removed R35: 100 kOhm 1%, Resistor_SMD:R_0402_1005Metric, symbol DioneyaMain:R35_ERJ-2RKF1003X
- removed R36: 22 Ohm 1%, Resistor_SMD:R_0402_1005Metric, symbol DioneyaMain:R36_ERJ-2RKF22R0X
- removed R37: 22 Ohm 1%, Resistor_SMD:R_0402_1005Metric, symbol DioneyaMain:R37_ERJ-2RKF22R0X
- removed R38: 1 kOhm 1%, Resistor_SMD:R_0402_1005Metric, symbol DioneyaMain:R38_ERJ-2RKF1001X
- removed R39: 0 Ohm, Resistor_SMD:R_0402_1005Metric, symbol DioneyaMain:R39_ERJ-2GE0R00X
- removed R4: 100 kOhm 1%, Resistor_SMD:R_0402_1005Metric, symbol DioneyaMain:R4_ERJ-2RKF1003X
- removed R40: 0 Ohm, Resistor_SMD:R_0402_1005Metric, symbol DioneyaMain:R40_ERJ-2GE0R00X
- removed R41: 1 kOhm 1%, Resistor_SMD:R_0402_1005Metric, symbol DioneyaMain:R41_ERJ-2RKF1001X
- removed R42: 0 Ohm, Resistor_SMD:R_0402_1005Metric, symbol DioneyaMain:R42_ERJ-2GE0R00X
- removed R43: 0 Ohm, Resistor_SMD:R_0402_1005Metric, symbol DioneyaMain:R43_ERJ-2GE0R00X
- removed R44: 47 kOhm 1%, Resistor_SMD:R_0402_1005Metric, symbol DioneyaMain:R44_ERJ-2RKF4702X
- removed R45: 100 kOhm 1%, Resistor_SMD:R_0402_1005Metric, symbol DioneyaMain:R45_ERJ-2RKF1003X
- removed R46: 10 kOhm 1%, Resistor_SMD:R_0402_1005Metric, symbol DioneyaMain:R46_ERJ-2RKF1002X
- removed R47: 100 kOhm 1%, Resistor_SMD:R_0402_1005Metric, symbol DioneyaMain:R47_ERJ-2RKF1003X
- removed R48: 10 kOhm 1%, Resistor_SMD:R_0402_1005Metric, symbol DioneyaMain:R48_ERJ-2RKF1002X
- removed R49: 10 kOhm 1%, Resistor_SMD:R_0402_1005Metric, symbol DioneyaMain:R49_ERJ-2RKF1002X
- removed R5: 100 kOhm 1%, Resistor_SMD:R_0402_1005Metric, symbol DioneyaMain:R5_ERJ-2RKF1003X
- removed R50: 0 Ohm, Resistor_SMD:R_0402_1005Metric, symbol DioneyaMain:R50_ERJ-2GE0R00X
- removed R51: 0 Ohm, Resistor_SMD:R_0402_1005Metric, symbol DioneyaMain:R51_ERJ-2GE0R00X
- removed R52: 0 Ohm, Resistor_SMD:R_0402_1005Metric, symbol DioneyaMain:R52_ERJ-2GE0R00X
- removed R53: 0 Ohm, Resistor_SMD:R_0402_1005Metric, symbol DioneyaMain:R53_ERJ-2GE0R00X
- removed R54: 0 Ohm, Resistor_SMD:R_0402_1005Metric, symbol DioneyaMain:R54_ERJ-2GE0R00X
- removed R55: 0 Ohm, Resistor_SMD:R_0402_1005Metric, symbol DioneyaMain:R55_ERJ-2GE0R00X
- removed R56: 22 Ohm 1%, Resistor_SMD:R_0402_1005Metric, symbol DioneyaMain:R56_ERJ-2RKF22R0X
- removed R57: 22 Ohm 1%, Resistor_SMD:R_0402_1005Metric, symbol DioneyaMain:R57_ERJ-2RKF22R0X
- removed R58: 22 Ohm 1%, Resistor_SMD:R_0402_1005Metric, symbol DioneyaMain:R58_ERJ-2RKF22R0X
- removed R59: 560 Ohm 5% 0.1 W, Resistor_SMD:R_0402_1005Metric, symbol DioneyaMain:R59_ERJ-2GEJ561X
- removed R6: 100 kOhm 1%, Resistor_SMD:R_0402_1005Metric, symbol DioneyaMain:R6_ERJ-2RKF1003X
- removed R60: 100 kOhm 5% 0.1 W, Resistor_SMD:R_0402_1005Metric, symbol DioneyaMain:R60_ERJ-2GEJ104X
- removed R61: 100 kOhm 5% 0.1 W, Resistor_SMD:R_0402_1005Metric, symbol DioneyaMain:R61_ERJ-2GEJ104X
- removed R62: 10 Ohm 5% 0.25 W, Resistor_SMD:R_1206_3216Metric, symbol DioneyaMain:R62_ERJ-8GEYJ100V
- removed R63: 100 kOhm 1%, Resistor_SMD:R_0402_1005Metric, symbol DioneyaMain:R63_ERJ-2RKF1003X
- removed R64: 100 kOhm 1%, Resistor_SMD:R_0402_1005Metric, symbol DioneyaMain:R64_ERJ-2RKF1003X
- removed R65: 100 kOhm 1%, Resistor_SMD:R_0402_1005Metric, symbol DioneyaMain:R65_ERJ-2RKF1003X
- removed R66: 100 kOhm 1%, Resistor_SMD:R_0402_1005Metric, symbol DioneyaMain:R66_ERJ-2RKF1003X
- removed R67: 10 kOhm 1%, Resistor_SMD:R_0402_1005Metric, symbol DioneyaMain:R67_ERJ-2RKF1002X
- removed R68: 10 kOhm 1%, Resistor_SMD:R_0402_1005Metric, symbol DioneyaMain:R68_ERJ-2RKF1002X
- removed R69: 22 Ohm 1%, Resistor_SMD:R_0402_1005Metric, symbol DioneyaMain:R69_ERJ-2RKF22R0X
- removed R7: 10 kOhm 1%, Resistor_SMD:R_0402_1005Metric, symbol DioneyaMain:R7_ERJ-2RKF1002X
- removed R70: 22 Ohm 1%, Resistor_SMD:R_0402_1005Metric, symbol DioneyaMain:R70_ERJ-2RKF22R0X
- removed R71: 22 Ohm 1%, Resistor_SMD:R_0402_1005Metric, symbol DioneyaMain:R71_ERJ-2RKF22R0X
- removed R72: 22 Ohm 1%, Resistor_SMD:R_0402_1005Metric, symbol DioneyaMain:R72_ERJ-2RKF22R0X
- removed R73: 0 Ohm, Resistor_SMD:R_0402_1005Metric, symbol DioneyaMain:R73_ERJ-2GE0R00X
- removed R74: 22 Ohm 1%, Resistor_SMD:R_0402_1005Metric, symbol DioneyaMain:R74_ERJ-2RKF22R0X
- removed R75: 22 Ohm 1%, Resistor_SMD:R_0402_1005Metric, symbol DioneyaMain:R75_ERJ-2RKF22R0X
- removed R76: 10 kOhm 1%, Resistor_SMD:R_0402_1005Metric, symbol DioneyaMain:R76_ERJ-2RKF1002X
- removed R77: 100 kOhm 1%, Resistor_SMD:R_0402_1005Metric, symbol DioneyaMain:R77_ERJ-2RKF1003X
- removed R78: 10 kOhm 1%, Resistor_SMD:R_0402_1005Metric, symbol DioneyaMain:R78_ERJ-2RKF1002X
- removed R79: 22 Ohm 1%, Resistor_SMD:R_0402_1005Metric, symbol DioneyaMain:R79_ERJ-2RKF22R0X
- removed R8: 22 Ohm 1%, Resistor_SMD:R_0402_1005Metric, symbol DioneyaMain:R8_ERJ-2RKF22R0X
- removed R80: 22 Ohm 1%, Resistor_SMD:R_0402_1005Metric, symbol DioneyaMain:R80_ERJ-2RKF22R0X
- removed R81: 22 Ohm 1%, Resistor_SMD:R_0402_1005Metric, symbol DioneyaMain:R81_ERJ-2RKF22R0X
- removed R82: 22 Ohm 1%, Resistor_SMD:R_0402_1005Metric, symbol DioneyaMain:R82_ERJ-2RKF22R0X
- removed R83: 22 Ohm 1%, Resistor_SMD:R_0402_1005Metric, symbol DioneyaMain:R83_ERJ-2RKF22R0X
- removed R84: 22 Ohm 1%, Resistor_SMD:R_0402_1005Metric, symbol DioneyaMain:R84_ERJ-2RKF22R0X
- removed R85: 10 kOhm 1%, Resistor_SMD:R_0402_1005Metric, symbol DioneyaMain:R85_ERJ-2RKF1002X
- removed R86: 10 kOhm 1%, Resistor_SMD:R_0402_1005Metric, symbol DioneyaMain:R86_ERJ-2RKF1002X
- removed R87: 10 kOhm 1%, Resistor_SMD:R_0402_1005Metric, symbol DioneyaMain:R87_ERJ-2RKF1002X
- removed R88: 10 kOhm 1%, Resistor_SMD:R_0402_1005Metric, symbol DioneyaMain:R88_ERJ-2RKF1002X
- removed R89: 10 kOhm 1%, Resistor_SMD:R_0402_1005Metric, symbol DioneyaMain:R89_ERJ-2RKF1002X
- removed R9: 22 Ohm 1%, Resistor_SMD:R_0402_1005Metric, symbol DioneyaMain:R9_ERJ-2RKF22R0X
- removed R90: 10 kOhm 1%, Resistor_SMD:R_0402_1005Metric, symbol DioneyaMain:R90_ERJ-2RKF1002X
- removed R91: 22 Ohm 1%, Resistor_SMD:R_0402_1005Metric, symbol DioneyaMain:R91_ERJ-2RKF22R0X
- removed R92: 22 Ohm 1%, Resistor_SMD:R_0402_1005Metric, symbol DioneyaMain:R92_ERJ-2RKF22R0X
- removed R93: 5.1 kOhm 1%, Resistor_SMD:R_0402_1005Metric, symbol DioneyaMain:R93_ERJ-2RKF5101X
- removed R94: 5.1 kOhm 1%, Resistor_SMD:R_0402_1005Metric, symbol DioneyaMain:R94_ERJ-2RKF5101X
- removed R95: 1 kOhm 1%, Resistor_SMD:R_0402_1005Metric, symbol DioneyaMain:R95_ERJ-2RKF1001X
- removed R96: 100 kOhm 1%, Resistor_SMD:R_0402_1005Metric, symbol DioneyaMain:R96_ERJ-2RKF1003X
- removed R97: 1 MOhm 1%, Resistor_SMD:R_0402_1005Metric, symbol DioneyaMain:R97_ERJ-2RKF1004X
- removed R98: 0 Ohm, Resistor_SMD:R_0402_1005Metric, symbol DioneyaMain:R98_ERJ-2GE0R00X
- removed R99: 10 kOhm 1%, Resistor_SMD:R_0402_1005Metric, symbol DioneyaMain:R99_ERJ-2RKF1002X
- removed TP_BLE_SWD: TEST_PADS, symbol DioneyaMain:TP_BLE_SWD_TEST_PADS
- removed TP_CELL_DBG: TEST_PADS, symbol DioneyaMain:TP_CELL_DBG_TEST_PADS
- removed TP_CELL_USB: TEST_PADS, symbol DioneyaMain:TP_CELL_USB_TEST_PADS
- removed TP_EOL: TEST_PADS, symbol DioneyaMain:TP_EOL_TEST_PADS
- removed TP_MCU_SWD: TEST_PADS, symbol DioneyaMain:TP_MCU_SWD_TEST_PADS
- removed U1: STM32U585VIT6Q, symbol DioneyaMain:U1_STM32U585VIT6Q
- removed U10: E22-900M22S, symbol DioneyaMain:U10_E22-900M22S
- removed U11: MDBT50Q-P1MV2, symbol DioneyaMain:U11_MDBT50Q-P1MV2
- removed U12: SDCIT2/32GB, symbol DioneyaMain:U12_SDCIT2_32GB
- removed U13: TS3A27518EPWR, symbol DioneyaMain:U13_TS3A27518EPWR
- removed U14: ESDALC6V1-5P6, symbol DioneyaMain:U14_ESDALC6V1-5P6
- removed U15: ESDALC6V1-5P6, symbol DioneyaMain:U15_ESDALC6V1-5P6
- removed U16: SN74AXC8T245PWR, symbol DioneyaMain:U16_SN74AXC8T245PWR
- removed U17: SN74LVC32APWR, symbol DioneyaMain:U17_SN74LVC32APWR
- removed U18: SN74AXC1T45DRLR, symbol DioneyaMain:U18_SN74AXC1T45DRLR
- removed U19: 4 channel 0.5 pF ESD, symbol DioneyaMain:U19_TPD4E05U06DQAR
- removed U2: W25Q512JVFIQ, symbol DioneyaMain:U2_W25Q512JVFIQ
- removed U20: 4 channel 0.5 pF ESD, symbol DioneyaMain:U20_TPD4E05U06DQAR
- removed U21: 4 channel 0.5 pF ESD, symbol DioneyaMain:U21_TPD4E05U06DQAR
- removed U22: 4 channel 0.5 pF ESD, symbol DioneyaMain:U22_TPD4E05U06DQAR
- removed U23: 4 channel 0.5 pF ESD, symbol DioneyaMain:U23_TPD4E05U06DQAR
- removed U24: 4 channel 0.5 pF ESD, symbol DioneyaMain:U24_TPD4E05U06DQAR
- removed U25: 2 channel 0.7 pF USB ESD, symbol DioneyaMain:U25_TPD2EUSB30DRTR
- removed U26: 2 channel 0.7 pF USB ESD, symbol DioneyaMain:U26_TPD2EUSB30DRTR
- removed U27: 4 channel 0.5 pF ESD, symbol DioneyaMain:U27_TPD4E05U06DQAR
- removed U3: LIS2DW12TR, symbol DioneyaMain:U3_LIS2DW12TR
- removed U4: STTS22HTR, symbol DioneyaMain:U4_STTS22HTR
- removed U5: Single rail-to-rail low-power op amp, symbol DioneyaMain:U5_LT6000IDCB_TRMPBF
- removed U6: Single non-inverting open-drain buffer, symbol DioneyaMain:U6_SN74LVC1G07DBVR
- removed U7: SN74AXC8T245PWR, symbol DioneyaMain:U7_SN74AXC8T245PWR
- removed U8: BG95-M3, symbol DioneyaMain:U8_BG95-M3
- removed U9: MAX-M10S-00B, symbol DioneyaMain:U9_MAX-M10S-00B
- removed X1: 32.768 kHz full-swing LVCMOS, symbol DioneyaMain:X1_SiT1552AI-JE-DCC-32.768D
Connections:
- no-connect marks 169 -> 0
Other:
- added sheet BLE module reset DFU and SWD (PCB-MAIN_07_BLE.kicad_sch)
- added sheet Cellular modem dual SIM and recovery (PCB-MAIN_05_CELLULAR.kicad_sch)
- added sheet GNSS timing antenna and supervisor (PCB-MAIN_04_GNSS.kicad_sch)
- added sheet LoRa radio control and conducted RF (PCB-MAIN_06_LORA.kicad_sch)
- added sheet MCU clocks reset and straps (PCB-MAIN_02_MCU.kicad_sch)
- added sheet PDM audio AAD and microphone harnesses (PCB-MAIN_03_AUDIO.kicad_sch)
- added sheet Power entry and rail interface (PCB-MAIN_01_POWER.kicad_sch)
- added sheet Storage sensors microSD and tamper (PCB-MAIN_08_STORAGE_SENSORS.kicad_sch)
- added sheet USB service debug and EOL fixture (PCB-MAIN_09_CONNECTORS_TEST.kicad_sch)
- note added: "Hierarchy-only engineering candidate. Signed Review-A pin/net authority is retained; routing, DRC, DFM, Review B and manufacture remain prohibited."
- title: Dioneya EVT-PRE-20 PCB-MAIN Rev.A -> Dioneya EVT-PRE-20 PCB-MAIN Rev.A - System overview

Commit message: hardware: fix PCB-MAIN hierarchy PDF layout
Other:
- title: Dioneya EVT-PRE-20 PCB-MAIN Rev.A - System overview -> Dioneya PCB-MAIN Rev.A - System overview
