File: hardware/kicad/native/PCB-MAIN/PCB-MAIN_01_POWER.kicad_sch (KiCad schematic)
At the start: 4 parts

Commit message: hardware: fix PCB-MAIN hierarchy PDF layout
Other:
- title: Dioneya EVT-PRE-20 PCB-MAIN Rev.A - Power entry and rail interface -> Dioneya PCB-MAIN Rev.A - Power
Changed lines of the file:
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@@
   (paper "A2")
   (title_block
-    (title "Dioneya EVT-PRE-20 PCB-MAIN Rev.A - Power entry and rail interface")
+    (title "Dioneya PCB-MAIN Rev.A - Power")
     (date "2026-09-16")
     (rev "A")
