File: hardware/kicad/native/PCB-MAIN/PCB-MAIN_02_MCU.kicad_sch (KiCad schematic)
At the start: 27 parts, among them U1 STM32U585VIT6Q, X1 32.768 kHz full-swing LVCMOS

Commit message: hardware: fix PCB-MAIN hierarchy PDF layout
Other:
- title: Dioneya EVT-PRE-20 PCB-MAIN Rev.A - MCU clocks reset and straps -> Dioneya PCB-MAIN Rev.A - MCU
Changed lines of the file:
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@@
   (paper "A2")
   (title_block
-    (title "Dioneya EVT-PRE-20 PCB-MAIN Rev.A - MCU clocks reset and straps")
+    (title "Dioneya PCB-MAIN Rev.A - MCU")
     (date "2026-09-16")
     (rev "A")
