File: hardware/kicad/native/PCB-MAIN/PCB-MAIN_03_AUDIO.kicad_sch (KiCad schematic)
At the start: 24 parts, among them U17 SN74LVC32APWR, U18 SN74AXC1T45DRLR, U19 4 channel 0.5 pF ESD, U20 4 channel 0.5 pF ESD, U21 4 channel 0.5 pF ESD, U22 4 channel 0.5 pF ESD, U7 SN74AXC8T245PWR

Commit message: hardware: fix PCB-MAIN hierarchy PDF layout
Other:
- title: Dioneya EVT-PRE-20 PCB-MAIN Rev.A - PDM audio AAD and microphone harnesses -> Dioneya PCB-MAIN Rev.A - PDM audio
Changed lines of the file:
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@@
   (paper "A2")
   (title_block
-    (title "Dioneya EVT-PRE-20 PCB-MAIN Rev.A - PDM audio AAD and microphone harnesses")
+    (title "Dioneya PCB-MAIN Rev.A - PDM audio")
     (date "2026-09-16")
     (rev "A")
