File: hardware/kicad/native/PCB-MAIN/PCB-MAIN_04_GNSS.kicad_sch (KiCad schematic)
At the start: 20 parts, among them J9 U.FL-R-SMT-1(60), Q4 Complementary N and P channel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, U5 Single rail-to-rail low-power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, U9 MAX-M10S-00B

Commit message: hardware: fix PCB-MAIN hierarchy PDF layout
Other:
- title: Dioneya EVT-PRE-20 PCB-MAIN Rev.A - GNSS timing antenna and supervisor -> Dioneya PCB-MAIN Rev.A - GNSS
Changed lines of the file:
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@@
   (paper "A2")
   (title_block
-    (title "Dioneya EVT-PRE-20 PCB-MAIN Rev.A - GNSS timing antenna and supervisor")
+    (title "Dioneya PCB-MAIN Rev.A - GNSS")
     (date "2026-09-16")
     (rev "A")
