File: hardware/kicad/native/PCB-MAIN/PCB-MAIN_05_CELLULAR.kicad_sch (KiCad schematic)
At the start: 81 parts, among them J6 2336582-1, J7 2336582-1, J8 U.FL-R-SMT-1(60), Q1 MMBT3904,215, Q2 MMBT3904,215, Q3 MMBT3904,215, U13 TS3A27518EPWR, U14 ESDALC6V1-5P6, U15 ESDALC6V1-5P6, U16 SN74AXC8T245PWR, U26 2 channel 0.7 pF USB ESD, U27 4 channel 0.5 pF ESD, U8 BG95-M3

Commit message: hardware: fix PCB-MAIN hierarchy PDF layout
Other:
- title: Dioneya EVT-PRE-20 PCB-MAIN Rev.A - Cellular modem dual SIM and recovery -> Dioneya PCB-MAIN Rev.A - Cellular + dual SIM
Changed lines of the file:
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@@
   (paper "A2")
   (title_block
-    (title "Dioneya EVT-PRE-20 PCB-MAIN Rev.A - Cellular modem dual SIM and recovery")
+    (title "Dioneya PCB-MAIN Rev.A - Cellular + dual SIM")
     (date "2026-09-16")
     (rev "A")
