File: hardware/kicad/native/PCB-MAIN/PCB-MAIN_06_LORA.kicad_sch (KiCad schematic)
At the start: 19 parts, among them J10 U.FL-R-SMT-1(60), U10 E22-900M22S

Commit message: hardware: fix PCB-MAIN hierarchy PDF layout
Other:
- title: Dioneya EVT-PRE-20 PCB-MAIN Rev.A - LoRa radio control and conducted RF -> Dioneya PCB-MAIN Rev.A - LoRa
Changed lines of the file:
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@@
   (paper "A2")
   (title_block
-    (title "Dioneya EVT-PRE-20 PCB-MAIN Rev.A - LoRa radio control and conducted RF")
+    (title "Dioneya PCB-MAIN Rev.A - LoRa")
     (date "2026-09-16")
     (rev "A")
