File: hardware/kicad/native/PCB-MAIN/PCB-MAIN_07_BLE.kicad_sch (KiCad schematic)
At the start: 11 parts, among them U11 MDBT50Q-P1MV2, U6 Single non-inverting open-dra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

Commit message: hardware: fix PCB-MAIN hierarchy PDF layout
Other:
- title: Dioneya EVT-PRE-20 PCB-MAIN Rev.A - BLE module reset DFU and SWD -> Dioneya PCB-MAIN Rev.A - BLE
Changed lines of the file:
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@@
   (paper "A2")
   (title_block
-    (title "Dioneya EVT-PRE-20 PCB-MAIN Rev.A - BLE module reset DFU and SWD")
+    (title "Dioneya PCB-MAIN Rev.A - BLE")
     (date "2026-09-16")
     (rev "A")
