File: hardware/kicad/native/PCB-MAIN/PCB-MAIN_08_STORAGE_SENSORS.kicad_sch (KiCad schematic)
At the start: 44 parts, among them J12 MEM2052-00-195-00-A, J13 504050-0291, U12 SDCIT2/32GB, U2 W25Q512JVFIQ, U23 4 channel 0.5 pF ESD, U24 4 channel 0.5 pF ESD, U3 LIS2DW12TR, U4 STTS22HTR

Commit message: hardware: fix PCB-MAIN hierarchy PDF layout
Other:
- title: Dioneya EVT-PRE-20 PCB-MAIN Rev.A - Storage sensors microSD and tamper -> Dioneya PCB-MAIN Rev.A - Storage + sensors
Changed lines of the file:
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@@
   (paper "A2")
   (title_block
-    (title "Dioneya EVT-PRE-20 PCB-MAIN Rev.A - Storage sensors microSD and tamper")
+    (title "Dioneya PCB-MAIN Rev.A - Storage + sensors")
     (date "2026-09-16")
     (rev "A")
