File: hardware/kicad/native/PCB-MAIN/PCB-MAIN_09_CONNECTORS_TEST.kicad_sch (KiCad schematic)
At the start: 18 parts, among them J11 USB4105-GF-A-120, U25 2 channel 0.7 pF USB ESD

Commit message: hardware: fix PCB-MAIN hierarchy PDF layout
Other:
- title: Dioneya EVT-PRE-20 PCB-MAIN Rev.A - USB service debug and EOL fixture -> Dioneya PCB-MAIN Rev.A - USB + debug
Changed lines of the file:
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@@
   (paper "A2")
   (title_block
-    (title "Dioneya EVT-PRE-20 PCB-MAIN Rev.A - USB service debug and EOL fixture")
+    (title "Dioneya PCB-MAIN Rev.A - USB + debug")
     (date "2026-09-16")
     (rev "A")
