File: hardware/kicad/native/PCB-PWR/PCB-PWR_01_INPUT_PROTECTION.kicad_sch (KiCad schematic)
At the start: 18 parts, among them J1 PWR_INPUT_43045-0213, Q1 CSD18540Q5B, U1 LM74700QDBVRQ1, U2 INA226AIDGSR

Commit message: hardware: apply PCB-PWR F1 value-only ECO
Parts:
- F1: value 0451005.MRL CANDIDATE -> 0451008.MRL
Changed lines of the file:
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@@
       (effects (font (size 0.85 0.85)))
     )
-    (property "Value" "0451005.MRL CANDIDATE" (id 1) (at 60.96 59.69 0)
+    (property "Value" "0451008.MRL" (id 1) (at 60.96 59.69 0)
       (effects (font (size 0.85 0.85)))
     )
