File: hardware/kicad/native/PCB-PWR/PCB-PWR_01_INPUT_PROTECTION.kicad_sch (KiCad schematic)
At the start: 18 parts, among them J1 PWR_INPUT_43045-0213, Q1 CSD18540Q5B, U1 LM74700QDBVRQ1, U2 INA226AIDGSR

Commit message: pcb-pwr: keep labels clear of connection wires
Other:
- title: Dioneya EVT-PRE-20 PCB-PWR Rev.A - Input protection and monitor -> Input protection + monitor
Changed lines of the file:
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@@
   (paper "A3")
   (title_block
-    (title "Dioneya EVT-PRE-20 PCB-PWR Rev.A - Input protection and monitor")
+    (title "Input protection + monitor")
     (date "2026-09-17")
     (rev "A")
@@
   )
   (label "LM74700_VCAP" (at 138.43 96.52 180)
-    (effects (font (size 1.1 1.1)))
+    (effects (font (size 1.1 1.1)) (justify bottom))
   )
   (label "VBAT_FUSED" (at 166.37 96.52 0)
-    (effects (font (size 1.1 1.1)))
+    (effects (font (size 1.1 1.1)) (justify bottom))
   )
   (label "VBAT_PROTECTED" (at 336.55 96.52 180)
-    (effects (font (size 1.1 1.1)))
+    (effects (font (size 1.1 1.1)) (justify bottom))
   )
   (label "GND_PWR" (at 364.49 96.52 0)
-    (effects (font (size 1.1 1.1)))
+    (effects (font (size 1.1 1.1)) (justify bottom))
   )
   (label "VBAT_SYS" (at 356.87 147.32 180)
-    (effects (font (size 1.1 1.1)))
+    (effects (font (size 1.1 1.1)) (justify bottom))
   )
   (label "GND_PWR" (at 384.81 147.32 0)
-    (effects (font (size 1.1 1.1)))
+    (effects (font (size 1.1 1.1)) (justify bottom))
   )
   (label "GND_PWR" (at 318.77 147.32 0)
-    (effects (font (size 1.1 1.1)))
+    (effects (font (size 1.1 1.1)) (justify bottom))
   )
   (label "VBAT_FUSED" (at 237.49 96.52 180)
-    (effects (font (size 1.1 1.1)))
+    (effects (font (size 1.1 1.1)) (justify bottom))
   )
   (label "GND_PWR" (at 265.43 96.52 0)
-    (effects (font (size 1.1 1.1)))
+    (effects (font (size 1.1 1.1)) (justify bottom))
   )
   (label "VBAT_FUSED" (at 41.91 96.52 180)
-    (effects (font (size 1.1 1.1)))
+    (effects (font (size 1.1 1.1)) (justify bottom))
   )
   (label "GND_PWR" (at 69.85 96.52 0)
-    (effects (font (size 1.1 1.1)))
+    (effects (font (size 1.1 1.1)) (justify bottom))
   )
   (label "VBAT_RAW" (at 138.43 48.26 180)
-    (effects (font (size 1.1 1.1)))
+    (effects (font (size 1.1 1.1)) (justify bottom))
   )
   (label "VBAT_FUSED" (at 166.37 48.26 0)
-    (effects (font (size 1.1 1.1)))
+    (effects (font (size 1.1 1.1)) (justify bottom))
   )
   (label "VBAT_RAW" (at 33.02 45.72 180)
-    (effects (font (size 1.1 1.1)))
+    (effects (font (size 1.1 1.1)) (justify bottom))
   )
   (label "GND_PWR" (at 33.02 50.8 180)
-    (effects (font (size 1.1 1.1)))
+    (effects (font (size 1.1 1.1)) (justify bottom))
   )
   (label "VBAT_FUSED" (at 325.12 43.18 180)
-    (effects (font (size 1.1 1.1)))
+    (effects (font (size 1.1 1.1)) (justify bottom))
   )
   (label "VBAT_FUSED" (at 325.12 48.26 180)
-    (effects (font (size 1.1 1.1)))
+    (effects (font (size 1.1 1.1)) (justify bottom))
   )
   (label "VBAT_FUSED" (at 325.12 53.34 180)
-    (effects (font (size 1.1 1.1)))
+    (effects (font (size 1.1 1.1)) (justify bottom))
   )
   (label "REV_GATE" (at 350.52 73.66 90)
-    (effects (font (size 1.1 1.1)))
+    (effects (font (size 1.1 1.1)) (justify bottom))
   )
   (label "VBAT_PROTECTED" (at 375.92 43.18 0)
-    (effects (font (size 1.1 1.1)))
+    (effects (font (size 1.1 1.1)) (justify bottom))
   )
   (label "VBAT_PROTECTED" (at 375.92 48.26 0)
-    (effects (font (size 1.1 1.1)))
+    (effects (font (size 1.1 1.1)) (justify bottom))
   )
   (label "VBAT_PROTECTED" (at 375.92 53.34 0)
-    (effects (font (size 1.1 1.1)))
+    (effects (font (size 1.1 1.1)) (justify bottom))
   )
   (label "VBAT_PROTECTED" (at 375.92 58.42 0)
-    (effects (font (size 1.1 1.1)))
+    (effects (font (size 1.1 1.1)) (justify bottom))
   )
   (label "VBAT_PROTECTED" (at 30.48 142.24 180)
-    (effects (font (size 1.1 1.1)))
+    (effects (font (size 1.1 1.1)) (justify bottom))
   )
   (label "VBAT_SYS" (at 106.68 142.24 0)
-    (effects (font (size 1.1 1.1)))
+    (effects (font (size 1.1 1.1)) (justify bottom))
   )
   (label "SHUNT_SOURCE_SENSE" (at 30.48 152.4 180)
-    (effects (font (size 1.1 1.1)))
+    (effects (font (size 1.1 1.1)) (justify bottom))
   )
   (label "SHUNT_LOAD_SENSE" (at 106.68 152.4 0)
-    (effects (font (size 1.1 1.1)))
+    (effects (font (size 1.1 1.1)) (justify bottom))
   )
   (label "VBAT_PROTECTED" (at 40.64 198.12 180)
-    (effects (font (size 1.1 1.1)))
+    (effects (font (size 1.1 1.1)) (justify bottom))
   )
   (label "SHUNT_SOURCE_SENSE" (at 137.16 198.12 180)
-    (effects (font (size 1.1 1.1)))
+    (effects (font (size 1.1 1.1)) (justify bottom))
   )
   (label "SHUNT_LOAD_SENSE" (at 236.22 198.12 180)
-    (effects (font (size 1.1 1.1)))
+    (effects (font (size 1.1 1.1)) (justify bottom))
   )
   (label "LM74700_VCAP" (at 223.52 55.88 180)
-    (effects (font (size 1.1 1.1)))
+    (effects (font (size 1.1 1.1)) (justify bottom))
   )
   (label "GND_PWR" (at 251.46 72.39 90)
-    (effects (font (size 1.1 1.1)))
+    (effects (font (size 1.1 1.1)) (justify bottom))
   )
   (label "VBAT_FUSED" (at 223.52 50.8 180)
-    (effects (font (size 1.1 1.1)))
+    (effects (font (size 1.1 1.1)) (justify bottom))
   )
   (label "VBAT_PROTECTED" (at 279.4 45.72 0)
-    (effects (font (size 1.1 1.1)))
+    (effects (font (size 1.1 1.1)) (justify bottom))
   )
   (label "REV_GATE" (at 279.4 50.8 0)
-    (effects (font (size 1.1 1.1)))
+    (effects (font (size 1.1 1.1)) (justify bottom))
   )
   (label "VBAT_FUSED" (at 223.52 45.72 180)
-    (effects (font (size 1.1 1.1)))
+    (effects (font (size 1.1 1.1)) (justify bottom))
   )
   (label "GND_PWR" (at 195.58 172.72 90)
-    (effects (font (size 1.1 1.1)))
+    (effects (font (size 1.1 1.1)) (justify bottom))
   )
   (label "GND_PWR" (at 205.74 172.72 90)
-    (effects (font (size 1.1 1.1)))
+    (effects (font (size 1.1 1.1)) (justify bottom))
   )
   (label "FAULT" (at 236.22 147.32 0)
-    (effects (font (size 1.1 1.1)))
+    (effects (font (size 1.1 1.1)) (justify bottom))
   )
   (label "I2C2_SDA" (at 175.26 152.4 180)
-    (effects (font (size 1.1 1.1)))
+    (effects (font (size 1.1 1.1)) (justify bottom))
   )
   (label "I2C2_SCL" (at 175.26 147.32 180)
-    (effects (font (size 1.1 1.1)))
+    (effects (font (size 1.1 1.1)) (justify bottom))
   )
   (label "3V3_DIGITAL" (at 205.74 121.92 270)
-    (effects (font (size 1.1 1.1)))
+    (effects (font (size 1.1 1.1)) (justify bottom))
   )
   (label "GND_PWR" (at 215.9 172.72 90)
-    (effects (font (size 1.1 1.1)))
+    (effects (font (size 1.1 1.1)) (justify bottom))
   )
   (label "VBAT_SYS" (at 175.26 142.24 180)
-    (effects (font (size 1.1 1.1)))
+    (effects (font (size 1.1 1.1)) (justify bottom))
   )
   (label "SHUNT_LOAD_SENSE" (at 236.22 139.7 0)
-    (effects (font (size 1.1 1.1)))
+    (effects (font (size 1.1 1.1)) (justify bottom))
   )
   (label "SHUNT_SOURCE_SENSE" (at 175.26 139.7 180)
-    (effects (font (size 1.1 1.1)))
+    (effects (font (size 1.1 1.1)) (justify bottom))
   )
   (hierarchical_label "VBAT_SYS" (shape passive) (at 236.22 238.76 180)
-    (effects (font (size 1.1 1.1)))
+    (effects (font (size 1.1 1.1)) (justify bottom))
   )
   (hierarchical_label "GND_PWR" (shape passive) (at 335.28 238.76 180)
-    (effects (font (size 1.1 1.1)))
+    (effects (font (size 1.1 1.1)) (justify bottom))
   )
   (hierarchical_label "3V3_DIGITAL" (shape passive) (at 290.83 147.32 180)
-    (effects (font (size 1.1 1.1)))
+    (effects (font (size 1.1 1.1)) (justify bottom))
   )
   (hierarchical_label "I2C2_SDA" (shape passive) (at 137.16 238.76 180)
-    (effects (font (size 1.1 1.1)))
+    (effects (font (size 1.1 1.1)) (justify bottom))
   )
   (hierarchical_label "FAULT" (shape passive) (at 335.28 198.12 180)
-    (effects (font (size 1.1 1.1)))
+    (effects (font (size 1.1 1.1)) (justify bottom))
   )
   (hierarchical_label "I2C2_SCL" (shape passive) (at 40.64 238.76 180)
-    (effects (font (size 1.1 1.1)))
+    (effects (font (size 1.1 1.1)) (justify bottom))
   )
   (symbol (lib_id "DioneyaPWR:ERC_SOURCE_FLAG") (at 251.46 238.76 0) (unit 1)
