File: hardware/kicad/candidates/PCB-MAIN-SIGNAL-HARD-NETS-001/PCB-MAIN_SIGNAL_HARD_NETS_BASE_REV_A.kicad_pcb (KiCad board)
At the start: 6 copper layers, 110 x 75 mm, 251 parts, among them J10 U.FL-R-SMT-1(60), J11 USB4105-GF-A-120, J12 MEM2052-00-195-00-A, J13 504050-0291, J6 2336582-1, J7 2336582-1, J8 U.FL-R-SMT-1(60), J9 U.FL-R-SMT-1(60), Q1 MMBT3904,215, Q2 MMBT3904,215, Q3 MMBT3904,215, Q4 Si1016X-T1-GE3, U1 STM32U585VIT6Q, U10 E22-900M22S, U11 MDBT50Q-P1MV2, U13 TS3A27518EPWR, U14 ESDALC6V1-5P6, U15 ESDALC6V1-5P6, U16 SN74AXC8T245PWR, U17 SN74LVC32APWR, U18 SN74AXC1T45DRLR, U19 TPD4E05U06DQAR, U2 W25Q512JVFIQ, U20 TPD4E05U06DQAR, U21 TPD4E05U06DQAR, U22 TPD4E05U06DQAR, U23 TPD4E05U06DQAR, U24 TPD4E05U06DQAR, U25 TPD2EUSB30DRTR, U26 TPD2EUSB30DRTR, U27 TPD4E05U06DQAR, U3 LIS2DW12TR, U4 STTS22HTR, U5 LT6000IDCB#TRMPBF, U6 SN74LVC1G07DBVR, U7 SN74AXC8T245PWR, U8 BG95-M3, U9 MAX-M10S-00B, X1 SiT1552AI-JE-DCC-32.768D

Commit message: hardware: apply PCB-MAIN hard signal routing subgate
Routing:
- net BLE_RX_U1: track 50.6 -> 0.00 mm
- net EN_MODEM: track 43.5 -> 0.00 mm, vias 1 -> 0
- net CELL_RX_U16: track 41.0 -> 0.00 mm
- net SD_D2_U1: track 35.9 -> 0.00 mm, vias 2 -> 0
- net SD_CMD_U1: track 31.0 -> 0.00 mm
- net NOR_IO2_U1: track 20.8 -> 0.00 mm, vias 2 -> 0
- net NOR_IO0_U1: track 20.0 -> 0.00 mm, vias 2 -> 0
- net BOOT0: track 19.0 -> 0.00 mm, vias 2 -> 0
