File: hardware/kicad/candidates/PCB-PWR-VBAT-RAW-ROUTING-003/PCB-PWR_VBAT_RAW_ROUTING_003_CANDIDATE_REV_A.kicad_pcb (KiCad board)
At the start: 4 copper layers, 90 x 60 mm, 66 parts, among them J1 43045-0213, J2 43045-1202, Q1 CSD18540Q5B, U1 LM74700QDBVRQ1, U2 INA226AIDGSR, U3 LMR604403SRAKR, U4 LMR604403SRAKR, U5 TPS7A2018PDBVR

Commit message: hardware: offset VBAT_RAW bridge for endpoint clearance
Routing:
- net VBAT_RAW: track 4.88 -> 2.90 mm
Changed lines of the file:
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@@
 	)
 	(segment
-		(start 6 31)
-		(end 10.6 29.357143)
+		(start 7.7 31.25)
+		(end 10.6 31.25)
 		(width 4)
 		(layer "F.Cu")
