File: hardware/kicad/candidates/PCB-PWR-AUTOROUTE-011/PCB-PWR_AUTOROUTE_011_CANDIDATE_REV_A.kicad_pcb (KiCad board)
At the start: 4 copper layers, 90 x 60 mm, 66 parts, among them J1 43045-0213, J2 43045-1202, Q1 CSD18540Q5B, U1 LM74700QDBVRQ1, U2 INA226AIDGSR, U3 LMR604403SRAKR, U4 LMR604403SRAKR, U5 TPS7A2018PDBVR

Commit message: apply: tools/apply_pcb_pwr_autoroute_candidate_rev_a.py
Routing:
- net BOOT_3V3: track 0.31 -> 1.60 mm
- net BOOT_3V8: track 0.31 -> 1.60 mm
- net VBAT_FUSED: track 45.9 -> 45.0 mm

Commit message: apply: tools/apply_pcb_pwr_autoroute_candidate_rev_a.py
Routing:
- net I2C2_SCL: track 40.9 -> 74.4 mm, vias 2 -> 3
- net VBAT_FUSED: track 45.0 -> 45.9 mm
