File: hardware/kicad/candidates/PCB-PWR-ECO-005/PCB-PWR_ECO_005_CANDIDATE_REV_A.kicad_pcb (KiCad board)
At the start: 4 copper layers, 90 x 60 mm, 66 parts, among them J1 43045-0213, J2 43045-1202, Q1 CSD18540Q5B, U1 LM74700QDBVRQ1, U2 INA226AIDGSR, U3 LMR604403SRAKR, U4 LMR604403SRAKR, U5 TPS7A2018PDBVR

Commit message: apply: tools/apply_pcb_pwr_eco_005_candidate_rev_a.py
Routing:
- net RT_3V8: track 23.8 -> 22.1 mm, vias 4 -> 3
Changed lines of the file:
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@@
 	)
 	(segment
-		(start 81.08 40)
-		(end 79.6065 41.4735)
+		(start 79.6065 41.4735)
+		(end 70.8572 41.4735)
 		(width 0.3)
 		(locked yes)
@@
 	)
 	(segment
+		(start 81.08 40)
+		(end 79.6065 41.4735)
+		(width 0.3)
+		(locked yes)
+		(layer "B.Cu")
+		(net 3)
+	)
+	(segment
 		(start 65.5104 37.669)
 		(end 53.3265 37.669)
@@
 	)
 	(segment
-		(start 79.6065 41.4735)
-		(end 70.8572 41.4735)
-		(width 0.3)
-		(locked yes)
-		(layer "B.Cu")
-		(net 3)
-	)
-	(segment
 		(start 70.8572 41.4735)
 		(end 66.6964 37.3127)
@@
 	)
 	(via
-		(at 74.5474 52.5526)
+		(at 73.85 52.95)
 		(size 0.6)
 		(drill 0.3)
 		(layers "F.Cu" "B.Cu")
+		(locked yes)
 		(net 11)
 	)
 	(via
-		(at 73.85 52.95)
+		(at 74.5474 52.5526)
 		(size 0.6)
 		(drill 0.3)
 		(layers "F.Cu" "B.Cu")
-		(locked yes)
 		(net 11)
 	)
@@
 	)
 	(via
-		(at 74.4 42.75)
+		(at 73.85 42.15)
 		(size 0.6)
 		(drill 0.3)
@@
 	)
 	(via
-		(at 73.85 42.15)
+		(at 74.4 42.75)
 		(size 0.6)
 		(drill 0.3)
@@
 	)
 	(via
+		(at 76.95 51.15)
+		(size 0.6)
+		(drill 0.3)
+		(layers "F.Cu" "B.Cu")
+		(locked yes)
+		(net 13)
+	)
+	(via
 		(at 10.45 45.45)
 		(size 0.6)
@@
 	)
 	(via
+		(at 74.35 48.15)
+		(size 0.6)
+		(drill 0.3)
+		(layers "F.Cu" "B.Cu")
+		(locked yes)
+		(net 13)
+	)
+	(via
 		(at 76.336037 40.078728)
 		(size 0.6)
@@
 	)
 	(via
-		(at 24.45 13.95)
+		(at 76.65 39.15)
 		(size 0.6)
 		(drill 0.3)
 		(layers "F.Cu" "B.Cu")
+		(locked yes)
 		(net 13)
 	)
 	(via
-		(at 38.45 6.95)
+		(at 24.45 13.95)
 		(size 0.6)
 		(drill 0.3)
@@
 	)
 	(via
-		(at 59.45 6.95)
+		(at 38.45 6.95)
 		(size 0.6)
 		(drill 0.3)
@@
 	)
 	(via
-		(at 48.95 3.45)
+		(at 59.45 6.95)
 		(size 0.6)
 		(drill 0.3)
@@
 	)
 	(via
-		(at 76.65 39.15)
+		(at 48.95 3.45)
 		(size 0.6)
 		(drill 0.3)
 		(layers "F.Cu" "B.Cu")
-		(locked yes)
 		(net 13)
 	)
@@
 	)
 	(via
-		(at 76.95 51.15)
-		(size 0.6)
-		(drill 0.3)
-		(layers "F.Cu" "B.Cu")
-		(locked yes)
-		(net 13)
-	)
-	(via
 		(at 24.45 10.45)
 		(size 0.6)
@@
 	)
 	(via
-		(at 74.55 49.05)
-		(size 0.6)
-		(drill 0.3)
-		(layers "F.Cu" "B.Cu")
-		(locked yes)
-		(net 13)
-	)
-	(via
 		(at 87.45 3.45)
 		(size 0.6)
@@
 	)
 	(via
-		(at 74.35 48.15)
-		(size 0.6)
-		(drill 0.3)
-		(layers "F.Cu" "B.Cu")
-		(locked yes)
-		(net 13)
-	)
-	(via
 		(at 87.45 45.45)
 		(size 0.6)
@@
 	)
 	(via
-		(at 73.75 48.75)
-		(size 0.6)
-		(drill 0.3)
-		(layers "F.Cu" "B.Cu")
-		(locked yes)
-		(net 13)
-	)
-	(via
 		(at 6.95 45.45)
 		(size 0.6)
@@
 	)
 	(via
+		(at 73.75 48.75)
+		(size 0.6)
+		(drill 0.3)
+		(layers "F.Cu" "B.Cu")
+		(locked yes)
+		(net 13)
+	)
+	(via
 		(at 45.45 6.95)
 		(size 0.6)
@@
 	)
 	(via
+		(at 74.55 49.05)
+		(size 0.6)
+		(drill 0.3)
+		(layers "F.Cu" "B.Cu")
+		(locked yes)
+		(net 13)
+	)
+	(via
 		(at 20.95 6.95)
 		(size 0.6)
@@
 	)
 	(segment
-		(start 54 12.3)
-		(end 53.6 11.5)
-		(width 0.2)
-		(locked yes)
-		(layer "F.Cu")
-		(net 23)
-	)
-	(segment
 		(start 53.8648 13.1)
 		(end 54 13.1)
@@
 	)
 	(segment
-		(start 54 12.9)
-		(end 54 12.3)
-		(width 0.2)
-		(locked yes)
-		(layer "F.Cu")
-		(net 23)
-	)
-	(segment
 		(start 53.825 13.1398)
 		(end 53.8648 13.1)
@@
 		(net 23)
 	)
-	(segment
-		(start 54 12.9)
-		(end 54 13.1)
-		(width 0.2006)
-		(layer "F.Cu")
-		(net 23)
-	)
 	(via
 		(at 49.35 15.15)
@@
 	)
 	(via
-		(at 53.6 11.5)
-		(size 0.6)
-		(drill 0.3)
-		(layers "F.Cu" "B.Cu")
-		(locked yes)
-		(net 23)
-	)
-	(via
 		(at 49.3725 18.2946)
 		(size 0.6)
@@
 	)
 	(zone
+		(net 10)
+		(net_name "GND_DIGITAL")
+		(layer "F.Cu")
+		(hatch edge 0.5)
+		(priority 14)
+		(connect_pads yes
+			(clearance 0.3)
+		)
+		(min_thickness 0.25)
+		(filled_areas_thickness no)
+		(fill yes
+			(thermal_gap 0.5)
+			(thermal_bridge_width 0.5)
+		)
+		(polygon
+			(pts
+				(xy 75.8 46.4) (xy 82.6 46.4) (xy 82.6 50.4) (xy 75.8 50.4)
+			)
+		)
+	)
+	(zone
 		(net 29)
 		(net_name "VBAT_PROTECTED")
@@
 			)
 		)
-	)
-	(zone
-		(net 10)
-		(net_name "GND_DIGITAL")
-		(layer "F.Cu")
-		(hatch edge 0.5)
-		(priority 14)
-		(connect_pads yes
-			(clearance 0.3)
-		)
-		(min_thickness 0.25)
-		(filled_areas_thickness no)
-		(fill yes
-			(thermal_gap 0.5)
-			(thermal_bridge_width 0.5)
-		)
-		(polygon
-			(pts
-				(xy 75.8 46.4) (xy 82.6 46.4) (xy 82.6 50.4) (xy 75.8 50.4)
-			)
-		)

Commit message: apply: tools/apply_pcb_pwr_eco_005_candidate_rev_a.py
Routing:
- net SHUNT_SOURCE_SENSE: track 47.3 -> 48.1 mm, vias 4 -> 3
