File: hardware/kicad/candidates/PCB-MAIN-GROUND-DOMAIN-ROUTING-002/PCB-MAIN_GROUND_DOMAIN_ROUTING_002_CANDIDATE_REV_A.kicad_pcb (KiCad board)
At the start: 6 copper layers, 110 x 75 mm, 251 parts, among them J10 U.FL-R-SMT-1(60), J11 USB4105-GF-A-120, J12 MEM2052-00-195-00-A, J13 504050-0291, J6 2336582-1, J7 2336582-1, J8 U.FL-R-SMT-1(60), J9 U.FL-R-SMT-1(60), Q1 MMBT3904,215, Q2 MMBT3904,215, Q3 MMBT3904,215, Q4 Si1016X-T1-GE3, U1 STM32U585VIT6Q, U10 E22-900M22S, U11 MDBT50Q-P1MV2, U13 TS3A27518EPWR, U14 ESDALC6V1-5P6, U15 ESDALC6V1-5P6, U16 SN74AXC8T245PWR, U17 SN74LVC32APWR, U18 SN74AXC1T45DRLR, U19 TPD4E05U06DQAR, U2 W25Q512JVFIQ, U20 TPD4E05U06DQAR, U21 TPD4E05U06DQAR, U22 TPD4E05U06DQAR, U23 TPD4E05U06DQAR, U24 TPD4E05U06DQAR, U25 TPD2EUSB30DRTR, U26 TPD2EUSB30DRTR, U27 TPD4E05U06DQAR, U3 LIS2DW12TR, U4 STTS22HTR, U5 LT6000IDCB#TRMPBF, U6 SN74LVC1G07DBVR, U7 SN74AXC8T245PWR, U8 BG95-M3, U9 MAX-M10S-00B, X1 SiT1552AI-JE-DCC-32.768D

Commit message: apply: tools/apply_pcb_main_ground_domain_routing_002_candidate_rev_a.py
Routing:
- net GND_MODEM: track 88.6 -> 101.2 mm
Changed lines of the file:
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@@
   (segment (start 38.5 25.5) (end 38.799999999999997 28.5) (width 0.1537) (layer "B.Cu") (net 33))
   (segment (start 38.799999999999997 28.5) (end 38.079999000000001 30) (width 0.1537) (layer "B.Cu") (net 33))
+  (segment (start 56.2250 29.1000) (end 57.9750 23.2250) (width 0.3) (layer "In3.Cu") (net 47))
+  (segment (start 57.9750 23.2250) (end 58.0750 21.5750) (width 0.3) (layer "In3.Cu") (net 47))
+  (segment (start 58.0750 21.5750) (end 60.1000 17.2250) (width 0.3) (layer "In3.Cu") (net 47))
   (via (at 8.199999999999999 50.149999999999999) (size 0.5) (drill 0.3) (layers "F.Cu" "B.Cu") (net 35))
   (via (at 8.699999999999999 52.640569415042094) (size 0.5) (drill 0.3) (layers "F.Cu" "B.Cu") (net 33))
