File: hardware/kicad/candidates/PCB-MAIN-INNER-REROUTE-003/PCB-MAIN_INNER_REROUTE_003_CANDIDATE_REV_A.kicad_pcb (KiCad board)
At the start: 6 copper layers, 110 x 75 mm, 251 parts, among them J10 U.FL-R-SMT-1(60), J11 USB4105-GF-A-120, J12 MEM2052-00-195-00-A, J13 504050-0291, J6 2336582-1, J7 2336582-1, J8 U.FL-R-SMT-1(60), J9 U.FL-R-SMT-1(60), Q1 MMBT3904,215, Q2 MMBT3904,215, Q3 MMBT3904,215, Q4 Si1016X-T1-GE3, U1 STM32U585VIT6Q, U10 E22-900M22S, U11 MDBT50Q-P1MV2, U13 TS3A27518EPWR, U14 ESDALC6V1-5P6, U15 ESDALC6V1-5P6, U16 SN74AXC8T245PWR, U17 SN74LVC32APWR, U18 SN74AXC1T45DRLR, U19 TPD4E05U06DQAR, U2 W25Q512JVFIQ, U20 TPD4E05U06DQAR, U21 TPD4E05U06DQAR, U22 TPD4E05U06DQAR, U23 TPD4E05U06DQAR, U24 TPD4E05U06DQAR, U25 TPD2EUSB30DRTR, U26 TPD2EUSB30DRTR, U27 TPD4E05U06DQAR, U3 LIS2DW12TR, U4 STTS22HTR, U5 LT6000IDCB#TRMPBF, U6 SN74LVC1G07DBVR, U7 SN74AXC8T245PWR, U8 BG95-M3, U9 MAX-M10S-00B, X1 SiT1552AI-JE-DCC-32.768D

Commit message: apply: tools/apply_pcb_main_inner_reroute_003_candidate_rev_a.py
Routing:
- net SD_D2_U1: vias 2 -> 0
- net NOR_IO3_U2: vias 3 -> 2
- net NOR_CLK_U1: vias 3 -> 2
Changed lines of the file:
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@@
     (property "DIONEA_PLACEMENT_SOURCE" "PCB_MAIN_PLACEMENT_REPACK_REV_A")
     (property "DIONEA_POPULATION" "FITTED")
-    (fp_text reference "R9" (at 0 -1.2) (layer "F.SilkS")
+    (fp_text reference "R9" (at 1.3 0 90) (layer "F.SilkS")
         (effects (font (size 0.8 0.8) (thickness 0.12)))
     )
@@
     (property "DIONEA_PLACEMENT_SOURCE" "PCB_MAIN_PLACEMENT_REPACK_REV_A")
     (property "DIONEA_POPULATION" "FITTED")
-    (fp_text reference "R10" (at 0 -1.2) (layer "F.SilkS")
+    (fp_text reference "R10" (at 1.3 0 90) (layer "F.SilkS")
         (effects (font (size 0.8 0.8) (thickness 0.12)))
     )
@@
     (property "DIONEA_PLACEMENT_SOURCE" "PCB_MAIN_PLACEMENT_REPACK_REV_A")
     (property "DIONEA_POPULATION" "FITTED")
-    (fp_text reference "R11" (at 0 -1.2) (layer "F.SilkS")
+    (fp_text reference "R11" (at 1.3 0 90) (layer "F.SilkS")
         (effects (font (size 0.8 0.8) (thickness 0.12)))
     )
@@
   (segment (start 54.225 15.975) (end 52.975 17.225) (width 0.15) (layer "F.Cu") (net 94))
   (segment (start 52.975 17.225) (end 52.975 17.975) (width 0.15) (layer "F.Cu") (net 94))
-  (via (at 52.975 17.975) (size 0.5) (drill 0.3) (layers "F.Cu" "B.Cu") (net 94))
   (segment (start 79.1 27.1) (end 80.6 27.1) (width 0.15) (layer "F.Cu") (net 95))
   (via (at 79.1 27.1) (size 0.5) (drill 0.3) (layers "F.Cu" "B.Cu") (net 95))
@@
   (via (at 69.975 27.725) (size 0.5) (drill 0.3) (layers "F.Cu" "B.Cu") (net 103))
   (via (at 41.475 27.85) (size 0.5) (drill 0.3) (layers "F.Cu" "B.Cu") (net 103))
-  (via (at 54.6 27.85) (size 0.5) (drill 0.3) (layers "F.Cu" "B.Cu") (net 103))
   (segment (start 54.6 27.85) (end 44.975 27.85) (width 0.15) (layer "B.Cu") (net 103))
   (segment (start 44.475 28.35) (end 41.975 28.35) (width 0.15) (layer "B.Cu") (net 103))
@@
   (segment (start 89.7 22.95) (end 89.2 22.45) (width 0.15) (layer "F.Cu") (net 136))
   (segment (start 56.95 23.45) (end 56.95 22.2) (width 0.15) (layer "F.Cu") (net 136))
-  (via (at 57.2 23.7) (size 0.5) (drill 0.3) (layers "F.Cu" "B.Cu") (net 136))
-  (via (at 89.2 21.7) (size 0.5) (drill 0.3) (layers "F.Cu" "B.Cu") (net 136))
   (segment (start 58.4125 67.975) (end 61.95 68.25) (width 0.1509) (layer "F.Cu") (net 57))
   (segment (start 61.95 68.25) (end 63.2 67) (width 0.1509) (layer "F.Cu") (net 57))
