File: hardware/kicad/candidates/PCB-ROUTING-004/PCB-MAIN_ROUTING_004_CANDIDATE_REV_A.kicad_pcb (KiCad board)
At the start: 6 copper layers, 110 x 75 mm, 251 parts, among them J10 U.FL-R-SMT-1(60), J11 USB4105-GF-A-120, J12 MEM2052-00-195-00-A, J13 504050-0291, J6 2336582-1, J7 2336582-1, J8 U.FL-R-SMT-1(60), J9 U.FL-R-SMT-1(60), Q1 MMBT3904,215, Q2 MMBT3904,215, Q3 MMBT3904,215, Q4 Si1016X-T1-GE3, U1 STM32U585VIT6Q, U10 E22-900M22S, U11 MDBT50Q-P1MV2, U13 TS3A27518EPWR, U14 ESDALC6V1-5P6, U15 ESDALC6V1-5P6, U16 SN74AXC8T245PWR, U17 SN74LVC32APWR, U18 SN74AXC1T45DRLR, U19 TPD4E05U06DQAR, U2 W25Q512JVFIQ, U20 TPD4E05U06DQAR, U21 TPD4E05U06DQAR, U22 TPD4E05U06DQAR, U23 TPD4E05U06DQAR, U24 TPD4E05U06DQAR, U25 TPD2EUSB30DRTR, U26 TPD2EUSB30DRTR, U27 TPD4E05U06DQAR, U3 LIS2DW12TR, U4 STTS22HTR, U5 LT6000IDCB#TRMPBF, U6 SN74LVC1G07DBVR, U7 SN74AXC8T245PWR, U8 BG95-M3, U9 MAX-M10S-00B, X1 SiT1552AI-JE-DCC-32.768D

Commit message: apply: tools/apply_pcb_main_routing_004_candidate_rev_a.py
Routing:
- net 3V3_DIGITAL: track 342.4 -> 0.00 mm, vias 22 -> 0
- net CELL_DBG_TXD_TP: track 75.7 -> 0.00 mm, vias 4 -> 0
- net EN_AUX: track 47.0 -> 0.00 mm, vias 1 -> 0
- net CELL_TX_U16: track 46.7 -> 0.00 mm, vias 8 -> 0
- net 3V8_MODEM: track 42.4 -> 0.00 mm, vias 1 -> 0
- net USB_VBUS_SENSE: track 41.6 -> 0.00 mm, vias 5 -> 0
- net SIM1_DET: track 40.6 -> 0.00 mm, vias 2 -> 0
- net CELL_USIM_CLK_1V8: track 38.2 -> 0.00 mm, vias 8 -> 0
- net CELL_USIM_RST_1V8: track 36.7 -> 0.00 mm, vias 6 -> 0
- net CELL_USIM_DATA_1V8: track 34.5 -> 0.00 mm, vias 4 -> 0
- net NRF_SWDIO: track 29.8 -> 0.00 mm, vias 1 -> 0
- net SD_D1_CARD: track 26.5 -> 0.00 mm, vias 3 -> 0
- net SD_D3_CARD: track 25.4 -> 0.00 mm, vias 3 -> 0
- net SD_D0_CARD: track 21.4 -> 0.00 mm, vias 2 -> 0
- net SD_DET: track 20.4 -> 0.00 mm, vias 3 -> 0
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
Commit message: apply: tools/apply_pcb_main_routing_004_candidate_rev_a.py
Routing:
- net 3V3_DIGITAL: track 0.00 -> 336.6 mm, vias 0 -> 21
- net SD_DET: track 0.00 -> 86.5 mm, vias 0 -> 3
- net 3V8_MODEM: track 0.00 -> 64.9 mm, vias 0 -> 4
- net SD_CK_CARD: track 22.8 -> 70.9 mm, vias 2 -> 4
- net EN_AUX: track 0.00 -> 46.0 mm, vias 0 -> 1
- net CELL_DBG_TXD_TP: track 0.00 -> 41.7 mm, vias 0 -> 4
- net CELL_DTR_U16: track 20.2 -> 60.0 mm, vias 2 -> 5
- net SIM_MUX_EN: track 0.00 -> 28.4 mm, vias 0 -> 4
- net NRF_SWDIO: track 0.00 -> 27.3 mm, vias 0 -> 1
- net NRF_SWCLK: track 0.00 -> 26.9 mm, vias 0 -> 1
- net SD_D0_CARD: track 0.00 -> 25.5 mm, vias 0 -> 4
- net SD_D1_CARD: track 0.00 -> 23.6 mm
- net LORA_NSS_U1: track 0.00 -> 21.0 mm, vias 0 -> 2
- net SD_CMD_CARD: track 19.2 -> 36.5 mm, vias 2 -> 3
- net SIM1_DATA_MUX: track 0.00 -> 14.7 mm, vias 0 -> 2
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
Commit message: apply: tools/apply_pcb_main_routing_004_candidate_rev_a.py
Routing:
- net SD_DET: track 86.5 -> 0.00 mm, vias 3 -> 0
- net 3V8_MODEM: track 64.9 -> 0.00 mm, vias 4 -> 0
- net EN_AUX: track 46.0 -> 0.00 mm, vias 1 -> 0
Changed lines of the file:
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@@
   (segment (start 91.8000 34.5500) (end 92.0750 34.2750) (width 0.3) (layer "F.Cu") (net 2))
   (segment (start 92.0750 34.2750) (end 92.0750 33.0000) (width 0.3) (layer "F.Cu") (net 2))
-  (segment (start 39.9816 51.0853) (end 39.4552 50.5589) (width 0.8) (layer "In3.Cu") (net 3))
-  (segment (start 39.4552 50.5589) (end 39.4552 39.4043) (width 0.8) (layer "In3.Cu") (net 3))
-  (segment (start 39.4552 39.4043) (end 36.4293 36.3784) (width 0.8) (layer "In3.Cu") (net 3))
-  (segment (start 36.4293 36.3784) (end 36.0362 36.3784) (width 0.8) (layer "In3.Cu") (net 3))
-  (segment (start 36.0362 36.3784) (end 35.5168 36.3784) (width 0.8) (layer "B.Cu") (net 3))
-  (segment (start 35.5168 36.3784) (end 26.2418 27.1034) (width 0.8) (layer "B.Cu") (net 3))
-  (segment (start 26.2418 27.1034) (end 18.1762 27.1034) (width 0.8) (layer "B.Cu") (net 3))
-  (segment (start 18.1762 27.1034) (end 16.9529 28.3267) (width 0.8) (layer "B.Cu") (net 3))
-  (segment (start 16.9529 28.3267) (end 15.6684 28.3267) (width 0.8) (layer "B.Cu") (net 3))
-  (segment (start 15.6684 28.3267) (end 14.7057 27.3640) (width 0.8) (layer "B.Cu") (net 3))
-  (segment (start 14.7057 27.3640) (end 12.9929 27.3640) (width 0.8) (layer "B.Cu") (net 3))
-  (segment (start 12.9929 27.3640) (end 12.4165 27.9404) (width 0.8) (layer "B.Cu") (net 3))
-  (segment (start 12.4165 27.9404) (end 10.4796 27.9404) (width 0.8) (layer "B.Cu") (net 3))
-  (segment (start 10.4796 27.9404) (end 8.9200 29.5000) (width 0.8) (layer "B.Cu") (net 3))
-  (segment (start 38.0369 24.7396) (end 37.8589 24.9176) (width 0.8) (layer "F.Cu") (net 3))
-  (segment (start 37.8589 24.9176) (end 37.8589 27.5644) (width 0.8) (layer "F.Cu") (net 3))
-  (segment (start 36.0362 36.3784) (end 36.0362 29.3871) (width 0.8) (layer "In3.Cu") (net 3))
-  (segment (start 36.0362 29.3871) (end 37.8589 27.5644) (width 0.8) (layer "In3.Cu") (net 3))
-  (segment (start 39.0000 52.0000) (end 39.0669 52.0000) (width 0.8) (layer "B.Cu") (net 3))
-  (segment (start 39.0669 52.0000) (end 39.9816 51.0853) (width 0.8) (layer "B.Cu") (net 3))
-  (segment (start 38.0369 24.7396) (end 38.0800 24.6965) (width 0.8) (layer "B.Cu") (net 3))
-  (segment (start 38.0800 24.6965) (end 38.0800 23.0000) (width 0.8) (layer "B.Cu") (net 3))
   (segment (start 37.8580 49.6280) (end 37.8580 34.7013) (width 0.8) (layer "F.Cu") (net 4))
   (segment (start 37.8580 34.7013) (end 37.6567 34.5000) (width 0.8) (layer "F.Cu") (net 4))
@@
   (segment (start 34.4478 16.3750) (end 33.6000 16.3750) (width 0.3) (layer "F.Cu") (net 41))
   (segment (start 33.1500 48.9000) (end 32.1348 48.9000) (width 0.3) (layer "F.Cu") (net 41))
-  (segment (start 42.6444 20.5328) (end 41.6577 21.5195) (width 0.15) (layer "B.Cu") (net 42))
-  (segment (start 41.6577 21.5195) (end 37.0136 21.5195) (width 0.15) (layer "B.Cu") (net 42))
-  (segment (start 37.0136 21.5195) (end 36.1143 20.6202) (width 0.15) (layer "B.Cu") (net 42))
-  (segment (start 36.1143 20.6202) (end 33.8992 20.6202) (width 0.15) (layer "B.Cu") (net 42))
-  (segment (start 33.8992 20.6202) (end 33.5128 21.0066) (width 0.15) (layer "B.Cu") (net 42))
-  (segment (start 33.5128 21.0066) (end 30.9167 21.0066) (width 0.15) (layer "B.Cu") (net 42))
-  (segment (start 30.9167 21.0066) (end 30.7618 21.1615) (width 0.15) (layer "B.Cu") (net 42))
-  (segment (start 30.7618 21.1615) (end 12.5815 21.1615) (width 0.15) (layer "B.Cu") (net 42))
-  (segment (start 12.5815 21.1615) (end 11.9200 20.5000) (width 0.15) (layer "B.Cu") (net 42))
-  (segment (start 53.0000 21.3733) (end 52.4171 21.3733) (width 0.15) (layer "F.Cu") (net 42))
-  (segment (start 52.4171 21.3733) (end 48.6795 17.6357) (width 0.15) (layer "F.Cu") (net 42))
-  (segment (start 48.6795 17.6357) (end 46.0389 17.6357) (width 0.15) (layer "F.Cu") (net 42))
-  (segment (start 46.0389 17.6357) (end 44.1797 19.4949) (width 0.15) (layer "F.Cu") (net 42))
-  (segment (start 44.1797 19.4949) (end 43.6823 19.4949) (width 0.15) (layer "F.Cu") (net 42))
-  (segment (start 43.6823 19.4949) (end 42.6444 20.5328) (width 0.15) (layer "F.Cu") (net 42))
-  (segment (start 53.0000 22.2500) (end 53.0000 21.3733) (width 0.15) (layer "F.Cu") (net 42))
   (segment (start 59.2456 56.5523) (end 59.2456 57.2485) (width 0.3) (layer "F.Cu") (net 48))
   (segment (start 59.2456 57.2485) (end 60.4221 58.4250) (width 0.3) (layer "F.Cu") (net 48))
@@
   (segment (start 91.9796 23.0954) (end 91.9796 24.1670) (width 0.15) (layer "F.Cu") (net 137))
   (segment (start 91.9796 24.1670) (end 91.6564 24.4902) (width 0.15) (layer "F.Cu") (net 137))
-  (segment (start 45.1267 27.0000) (end 45.1267 26.2600) (width 0.15) (layer "F.Cu") (net 139))
-  (segment (start 45.1267 26.2600) (end 45.3829 26.0038) (width 0.15) (layer "F.Cu") (net 139))
-  (segment (start 45.3829 26.0038) (end 45.3829 23.5540) (width 0.15) (layer "B.Cu") (net 139))
-  (segment (start 45.3829 23.5540) (end 43.8903 22.0614) (width 0.15) (layer "B.Cu") (net 139))
-  (segment (start 43.8903 22.0614) (end 43.8903 21.0249) (width 0.15) (layer "B.Cu") (net 139))
-  (segment (start 43.8903 21.0249) (end 42.8464 19.9810) (width 0.15) (layer "B.Cu") (net 139))
-  (segment (start 42.8464 19.9810) (end 42.4309 19.9810) (width 0.15) (layer "B.Cu") (net 139))
-  (segment (start 42.4309 19.9810) (end 41.2441 21.1678) (width 0.15) (layer "B.Cu") (net 139))
-  (segment (start 41.2441 21.1678) (end 37.9945 21.1678) (width 0.15) (layer "B.Cu") (net 139))
-  (segment (start 37.9945 21.1678) (end 37.6086 20.7819) (width 0.15) (layer "B.Cu") (net 139))
-  (segment (start 37.6086 20.7819) (end 37.6086 20.3921) (width 0.15) (layer "B.Cu") (net 139))
-  (segment (start 37.6086 20.3921) (end 45.0164 12.9843) (width 0.15) (layer "B.Cu") (net 139))
-  (segment (start 45.0164 12.9843) (end 69.9845 12.9843) (width 0.15) (layer "B.Cu") (net 139))
-  (segment (start 69.9845 12.9843) (end 78.7818 21.7816) (width 0.15) (layer "B.Cu") (net 139))
-  (segment (start 78.7818 21.7816) (end 80.7475 21.7816) (width 0.15) (layer "B.Cu") (net 139))
-  (segment (start 83.8750 24.8384) (end 81.6882 24.8384) (width 0.15) (layer "B.Cu") (net 139))
-  (segment (start 81.6882 24.8384) (end 80.7475 23.8977) (width 0.15) (layer "B.Cu") (net 139))
-  (segment (start 80.7475 23.8977) (end 80.7475 21.7816) (width 0.15) (layer "B.Cu") (net 139))
-  (segment (start 83.3250 23.0000) (end 83.8750 23.5500) (width 0.15) (layer "F.Cu") (net 139))
-  (segment (start 83.8750 23.5500) (end 83.8750 24.8384) (width 0.15) (layer "F.Cu") (net 139))
-  (segment (start 80.7475 21.7816) (end 84.5918 21.7816) (width 0.15) (layer "B.Cu") (net 139))
-  (segment (start 84.5918 21.7816) (end 85.0933 21.2801) (width 0.15) (layer "B.Cu") (net 139))
-  (segment (start 44.2500 27.0000) (end 45.1267 27.0000) (width 0.15) (layer "F.Cu") (net 139))
-  (segment (start 86.2908 21.0700) (end 86.7208 21.5000) (width 0.15) (layer "F.Cu") (net 139))
-  (segment (start 86.7208 21.5000) (end 87.5825 21.5000) (width 0.15) (layer "F.Cu") (net 139))
-  (segment (start 90.5850 17.7200) (end 88.5843 17.7200) (width 0.15) (layer "F.Cu") (net 139))
-  (segment (start 88.5843 17.7200) (end 86.2908 20.0135) (width 0.15) (layer "F.Cu") (net 139))
-  (segment (start 86.2908 20.0135) (end 86.2908 21.0700) (width 0.15) (layer "F.Cu") (net 139))
-  (segment (start 86.2908 21.0700) (end 85.3034 21.0700) (width 0.15) (layer "F.Cu") (net 139))
-  (segment (start 85.3034 21.0700) (end 85.0933 21.2801) (width 0.15) (layer "F.Cu") (net 139))
   (segment (start 23.5767 20.0000) (end 23.6376 20.0609) (width 0.15) (layer "F.Cu") (net 140))
   (segment (start 23.6376 20.0609) (end 23.7545 20.0609) (width 0.15) (layer "F.Cu") (net 140))
@@
   (via (at 35.3116 18.9750) (size 0.5) (drill 0.3) (layers "F.Cu" "B.Cu") (net 2))
   (via (at 35.6184 21.6960) (size 0.5) (drill 0.3) (layers "F.Cu" "B.Cu") (net 2))
-  (via (at 36.0362 36.3784) (size 0.5) (drill 0.3) (layers "F.Cu" "B.Cu") (net 3))
-  (via (at 38.0369 24.7396) (size 0.5) (drill 0.3) (layers "F.Cu" "B.Cu") (net 3))
-  (via (at 37.8589 27.5644) (size 0.5) (drill 0.3) (layers "F.Cu" "B.Cu") (net 3))
-  (via (at 39.9816 51.0853) (size 0.5) (drill 0.3) (layers "F.Cu" "B.Cu") (net 3))
   (via (at 34.1964 61.6000) (size 0.5) (drill 0.3) (layers "F.Cu" "B.Cu") (net 4))
   (via (at 37.8580 49.6280) (size 0.5) (drill 0.3) (layers "F.Cu" "B.Cu") (net 4))
@@
   (via (at 34.8032 21.5750) (size 0.5) (drill 0.3) (layers "F.Cu" "B.Cu") (net 41))
   (via (at 34.9327 19.6250) (size 0.5) (drill 0.3) (layers "F.Cu" "B.Cu") (net 41))
-  (via (at 42.6444 20.5328) (size 0.5) (drill 0.3) (layers "F.Cu" "B.Cu") (net 42))
   (via (at 53.9732 55.4601) (size 0.5) (drill 0.3) (layers "F.Cu" "B.Cu") (net 49))
   (via (at 62.0818 55.4601) (size 0.5) (drill 0.3) (layers "F.Cu" "B.Cu") (net 49))
@@
   (via (at 89.2392 25.2475) (size 0.5) (drill 0.3) (layers "F.Cu" "B.Cu") (net 137))
   (via (at 91.6564 24.4902) (size 0.5) (drill 0.3) (layers "F.Cu" "B.Cu") (net 137))
-  (via (at 83.8750 24.8384) (size 0.5) (drill 0.3) (layers "F.Cu" "B.Cu") (net 139))
-  (via (at 45.3829 26.0038) (size 0.5) (drill 0.3) (layers "F.Cu" "B.Cu") (net 139))
-  (via (at 85.0933 21.2801) (size 0.5) (drill 0.3) (layers "F.Cu" "B.Cu") (net 139))
   (via (at 23.7545 20.0609) (size 0.5) (drill 0.3) (layers "F.Cu" "B.Cu") (net 140))
   (via (at 20.9938 15.3762) (size 0.5) (drill 0.3) (layers "F.Cu" "B.Cu") (net 140))
