File: hardware/kicad/candidates/PCB-ROUTING-005/PCB-MAIN_ROUTING_005_CANDIDATE_REV_A.kicad_pcb (KiCad board)
At the start: 6 copper layers, 110 x 75 mm, 251 parts, among them J10 U.FL-R-SMT-1(60), J11 USB4105-GF-A-120, J12 MEM2052-00-195-00-A, J13 504050-0291, J6 2336582-1, J7 2336582-1, J8 U.FL-R-SMT-1(60), J9 U.FL-R-SMT-1(60), Q1 MMBT3904,215, Q2 MMBT3904,215, Q3 MMBT3904,215, Q4 Si1016X-T1-GE3, U1 STM32U585VIT6Q, U10 E22-900M22S, U11 MDBT50Q-P1MV2, U13 TS3A27518EPWR, U14 ESDALC6V1-5P6, U15 ESDALC6V1-5P6, U16 SN74AXC8T245PWR, U17 SN74LVC32APWR, U18 SN74AXC1T45DRLR, U19 TPD4E05U06DQAR, U2 W25Q512JVFIQ, U20 TPD4E05U06DQAR, U21 TPD4E05U06DQAR, U22 TPD4E05U06DQAR, U23 TPD4E05U06DQAR, U24 TPD4E05U06DQAR, U25 TPD2EUSB30DRTR, U26 TPD2EUSB30DRTR, U27 TPD4E05U06DQAR, U3 LIS2DW12TR, U4 STTS22HTR, U5 LT6000IDCB#TRMPBF, U6 SN74LVC1G07DBVR, U7 SN74AXC8T245PWR, U8 BG95-M3, U9 MAX-M10S-00B, X1 SiT1552AI-JE-DCC-32.768D

Commit message: apply: tools/apply_pcb_main_routing_005_candidate_rev_a.py
Routing:
- net GNSS_ANT_OFF_N: track 26.1 -> 0.00 mm, vias 2 -> 0
- net VCORE_1V1: track 16.3 -> 0.00 mm, vias 2 -> 0
Changed lines of the file:
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@@
   (segment (start 61.7775 27.8606) (end 62.5356 27.8606) (width 0.3) (layer "F.Cu") (net 2))
   (segment (start 62.5356 27.8606) (end 63.1750 28.5000) (width 0.3) (layer "F.Cu") (net 2))
-  (segment (start 60.3620 65.0000) (end 60.8777 65.0000) (width 0.15) (layer "F.Cu") (net 52))
-  (segment (start 51.1072 55.3046) (end 56.5180 60.7154) (width 0.15) (layer "F.Cu") (net 52))
-  (segment (start 56.5180 60.7154) (end 59.6526 60.7154) (width 0.15) (layer "F.Cu") (net 52))
-  (segment (start 59.6526 60.7154) (end 60.8777 61.9405) (width 0.15) (layer "F.Cu") (net 52))
-  (segment (start 60.8777 61.9405) (end 60.8777 65.0000) (width 0.15) (layer "F.Cu") (net 52))
-  (segment (start 52.6908 49.9999) (end 52.2300 50.4607) (width 0.15) (layer "B.Cu") (net 52))
-  (segment (start 52.2300 50.4607) (end 52.2300 54.1818) (width 0.15) (layer "B.Cu") (net 52))
-  (segment (start 52.2300 54.1818) (end 51.1072 55.3046) (width 0.15) (layer "B.Cu") (net 52))
-  (segment (start 54.6000 53.2500) (end 54.6000 51.9091) (width 0.15) (layer "F.Cu") (net 52))
-  (segment (start 54.6000 51.9091) (end 52.6908 49.9999) (width 0.15) (layer "F.Cu") (net 52))
   (segment (start 48.5000 37.7500) (end 48.5000 40.3968) (width 0.15) (layer "F.Cu") (net 74))
   (segment (start 48.5000 40.3968) (end 48.0368 40.8600) (width 0.15) (layer "F.Cu") (net 74))
@@
   (segment (start 85.0933 21.2801) (end 85.3132 21.5000) (width 0.15) (layer "F.Cu") (net 139))
   (segment (start 85.3132 21.5000) (end 87.5825 21.5000) (width 0.15) (layer "F.Cu") (net 139))
-  (segment (start 59.3228 39.5316) (end 59.2475 39.6069) (width 0.3) (layer "F.Cu") (net 185))
-  (segment (start 59.2475 39.6069) (end 54.2696 39.6069) (width 0.3) (layer "F.Cu") (net 185))
-  (segment (start 54.2696 39.6069) (end 53.4250 40.4515) (width 0.3) (layer "F.Cu") (net 185))
-  (segment (start 53.4250 40.4515) (end 53.4250 40.7500) (width 0.3) (layer "F.Cu") (net 185))
-  (segment (start 61.6277 32.7783) (end 59.5488 34.8572) (width 0.3) (layer "In3.Cu") (net 185))
-  (segment (start 59.5488 34.8572) (end 59.5488 39.3056) (width 0.3) (layer "In3.Cu") (net 185))
-  (segment (start 59.5488 39.3056) (end 59.3228 39.5316) (width 0.3) (layer "In3.Cu") (net 185))
-  (segment (start 61.4250 33.5000) (end 61.4250 32.9810) (width 0.3) (layer "F.Cu") (net 185))
-  (segment (start 61.4250 32.9810) (end 61.6277 32.7783) (width 0.3) (layer "F.Cu") (net 185))
-  (segment (start 61.4250 33.5000) (end 61.4250 34.7500) (width 0.3) (layer "F.Cu") (net 185))
   (via (at 8.199999999999999 50.149999999999999) (size 0.5) (drill 0.3) (layers "F.Cu" "B.Cu") (net 35))
   (via (at 8.699999999999999 52.640569415042094) (size 0.5) (drill 0.3) (layers "F.Cu" "B.Cu") (net 33))
@@
   (via (at 41.4674 32.1324) (size 0.5) (drill 0.3) (layers "F.Cu" "B.Cu") (net 186))
   (via (at 40.9333 34.6989) (size 0.5) (drill 0.3) (layers "F.Cu" "B.Cu") (net 186))
-  (via (at 51.1072 55.3046) (size 0.5) (drill 0.3) (layers "F.Cu" "B.Cu") (net 52))
-  (via (at 52.6908 49.9999) (size 0.5) (drill 0.3) (layers "F.Cu" "B.Cu") (net 52))
   (via (at 51.0115 19.8778) (size 0.5) (drill 0.3) (layers "F.Cu" "B.Cu") (net 128))
   (via (at 44.8045 19.7354) (size 0.5) (drill 0.3) (layers "F.Cu" "B.Cu") (net 128))
   (via (at 85.0933 21.2801) (size 0.5) (drill 0.3) (layers "F.Cu" "B.Cu") (net 139))
   (via (at 83.8750 24.8217) (size 0.5) (drill 0.3) (layers "F.Cu" "B.Cu") (net 139))
-  (via (at 59.3228 39.5316) (size 0.5) (drill 0.3) (layers "F.Cu" "B.Cu") (net 185))
-  (via (at 61.6277 32.7783) (size 0.5) (drill 0.3) (layers "F.Cu" "B.Cu") (net 185))
   (zone (net 0) (net_name "") (layers "F.Cu" "In1.Cu" "In2.Cu" "In3.Cu" "In4.Cu" "B.Cu") (name "PCB_MAIN_H1_NO_COPPER_D8_AUTHORITY") (hatch edge 0.5)
     (connect_pads (clearance 0))
