File: hardware/kicad/candidates/PCB-ROUTING-G/PCB-MAIN_ROUTING_G_CANDIDATE_REV_A.kicad_pcb (KiCad board)
At the start: 6 copper layers, 110 x 75 mm, 251 parts, among them J10 U.FL-R-SMT-1(60), J11 USB4105-GF-A-120, J12 MEM2052-00-195-00-A, J13 504050-0291, J6 2336582-1, J7 2336582-1, J8 U.FL-R-SMT-1(60), J9 U.FL-R-SMT-1(60), Q1 MMBT3904,215, Q2 MMBT3904,215, Q3 MMBT3904,215, Q4 Si1016X-T1-GE3, U1 STM32U585VIT6Q, U10 E22-900M22S, U11 MDBT50Q-P1MV2, U13 TS3A27518EPWR, U14 ESDALC6V1-5P6, U15 ESDALC6V1-5P6, U16 SN74AXC8T245PWR, U17 SN74LVC32APWR, U18 SN74AXC1T45DRLR, U19 TPD4E05U06DQAR, U2 W25Q512JVFIQ, U20 TPD4E05U06DQAR, U21 TPD4E05U06DQAR, U22 TPD4E05U06DQAR, U23 TPD4E05U06DQAR, U24 TPD4E05U06DQAR, U25 TPD2EUSB30DRTR, U26 TPD2EUSB30DRTR, U27 TPD4E05U06DQAR, U3 LIS2DW12TR, U4 STTS22HTR, U5 LT6000IDCB#TRMPBF, U6 SN74LVC1G07DBVR, U7 SN74AXC8T245PWR, U8 BG95-M3, U9 MAX-M10S-00B, X1 SiT1552AI-JE-DCC-32.768D

Commit message: apply: tools/apply_pcb_main_routing_g_candidate_rev_a.py
Routing:
- net 1V8_MIC: track 212.8 -> 0.00 mm, vias 5 -> 0
- net AAD_CFG_1V8_FANOUT: track 173.1 -> 0.00 mm, vias 3 -> 0
- net AAD_CFG: track 79.4 -> 0.00 mm, vias 10 -> 0
- net PDM_DATA1_1V8: track 58.5 -> 0.00 mm, vias 4 -> 0
- net CELL_RI_U16: track 49.2 -> 0.00 mm, vias 6 -> 0
- net GNSS_ANT_SHORT_N: track 48.2 -> 0.00 mm, vias 3 -> 0
- net SIM_MUX_EN: track 31.2 -> 0.00 mm, vias 2 -> 0
- net LORA_NSS_U1: track 30.5 -> 0.00 mm, vias 4 -> 0
- net GNSS_ANT_GATE: track 24.9 -> 0.00 mm, vias 2 -> 0
- net CELL_USB_BOOT_1V8: track 21.5 -> 0.00 mm
